Commit message: Fix the slider name from 'slider_left' to 'slider_right'
When I tried to load the URDF file on MuJoCo, it failed with the
following error message:

    Duplicated slider name "slider_left"

It turned out that the issue was the right slider being wrongly
tagged as 'slider_left' (not 'slider_right'). Fix it thusly.

Signed-off-by: Fujimoto Seiji <fujimoto@ceptord.net>

File: openarm_grip_description/urdf/openarm_grip.urdf (robot description, URDF)
Before this commit: robot openarm_grip, 11 links, 9 joints
Joints:
- added joint slider_right: type prismatic, parent grip_attach_1, child right_jaw_1, origin xyz=0.0775 -0.121655 0.012086 rpy=0 0 0, axis 1.0 -0.0 0.0, limit lower=-0.0455 upper=0.0 effort=100 velocity=1.0
- joint slider_left: axis 1.0 -0.0 0.0 -> -1.0 0.0 -0.0; child right_jaw_1 -> left_jaw_1; origin xyz=0.0775 -0.121655 0.012086 rpy=0 0 0 -> xyz=-0.0775 -0.121655 0.012086 rpy=0 0 0

File: openarm_grip_description/urdf/openarm_grip.xacro (robot description, xacro)
@@ -265,5 +265,5 @@
   <limit upper="0.0" lower="-0.0455" effort="100" velocity="1.0" acceleration="0.5"/>
 </joint>
-<joint name="slider_left" type="prismatic">
+<joint name="slider_right" type="prismatic">
   <origin xyz="0.0775 -0.121655 0.012086" rpy="0 0 0"/>
   <parent link="grip_attach_1"/>

Commit message: Add mimic tag to control left and right gripper equally

File: openarm_grip_description/urdf/openarm_grip.urdf (robot description, URDF)
Before this commit: robot openarm_grip, 11 links, 10 joints
Joints:
- joint slider_right: mimic (none) -> joint=slider_left

File: openarm_grip_description/urdf/openarm_grip.xacro (robot description, xacro)
@@ -271,4 +271,5 @@
   <axis xyz="1.0 -0.0 0.0"/>
   <limit upper="0.0" lower="-0.0455" effort="100" velocity="1.0" acceleration="0.5"/>
+  <mimic joint="slider_left"/>
 </joint>
 </robot>

Commit message: Update urdf for better gazebo compatibility

File: openarm_grip_description/urdf/openarm_grip.urdf (robot description, URDF)
Before this commit: robot openarm_grip, 11 links, 10 joints
Links:
- removed link dummy
- added link world
Joints:
- removed joint dummy_joint
- added joint world_joint: type fixed, parent world, child base_link, origin xyz=0.0 0.0 0.0 rpy=0.0 0.0 0.0

File: openarm_grip_description/urdf/openarm_grip.xacro (robot description, xacro)
@@ -1,10 +1,10 @@
 <?xml version="1.0" ?>
 <robot name="openarm_grip" xmlns:xacro="http://www.ros.org/wiki/xacro">
-<xacro:include filename="$(find openarm_grip_description)/urdf/materials.xacro" />
-<xacro:include filename="$(find openarm_grip_description)/urdf/openarm_grip.trans" />
-<xacro:include filename="$(find openarm_grip_description)/urdf/openarm_grip.gazebo" />
-<link name="dummy"/>
-<joint name="dummy_joint" type="fixed">
-  <parent link="dummy"/>
+<xacro:include filename="package://openarm_grip_description/urdf/materials.xacro" />
+<xacro:include filename="package://openarm_grip_description/urdf/openarm_grip.trans" />
+<xacro:include filename="package://openarm_grip_description/urdf/openarm_grip.gazebo" />
+<link name="world"/>
+<joint name="world_joint" type="fixed">
+  <parent link="world"/>
   <child link="base_link"/>
   <origin xyz="0.0 0.0 0.0" rpy="0.0 0.0 0.0"/>
@@ -216,4 +216,5 @@
   <axis xyz="0.0 0.0 1.0"/>
   <limit upper="2.356194" lower="-2.356194" effort="100" velocity="1.0" acceleration="0.5"/>
+  <dynamics damping="1.0" friction="1.0"/>
 </joint>
 <joint name="rev2" type="revolute">
@@ -223,4 +224,5 @@
   <axis xyz="-1.0 -0.0 0.0"/>
   <limit upper="0.0" lower="-3.054326" effort="100" velocity="1.0" acceleration="0.5"/>
+  <dynamics damping="1.0" friction="1.0"/>
 </joint>
 <joint name="rev3" type="revolute">
@@ -230,4 +232,5 @@
   <axis xyz="-0.0 0.986291 0.165017"/>
   <limit upper="2.094395" lower="-2.094395" effort="100" velocity="1.0" acceleration="0.5"/>
+  <dynamics damping="1.0" friction="1.0"/>
 </joint>
 <joint name="rev4" type="revolute">
@@ -237,4 +240,5 @@
   <axis xyz="1.0 0.0 0.0"/>
   <limit upper="0.0" lower="-3.141593" effort="100" velocity="1.0" acceleration="0.5"/>
+  <dynamics damping="1.0" friction="1.0"/>
 </joint>
 <joint name="rev5" type="revolute">
@@ -244,4 +248,5 @@
   <axis xyz="0.0 -0.980588 0.196078"/>
   <limit upper="2.094395" lower="-2.094395" effort="100" velocity="1.0" acceleration="0.5"/>
+  <dynamics damping="1.0" friction="1.0"/>
 </joint>
 <joint name="rev6" type="revolute">
@@ -251,4 +256,5 @@
   <axis xyz="-1.0 0.0 -0.0"/>
   <limit upper="1.570796" lower="-1.570796" effort="100" velocity="1.0" acceleration="0.5"/>
+  <dynamics damping="1.0" friction="1.0"/>
 </joint>
 <joint name="rev7" type="continuous">
@@ -257,4 +263,5 @@
   <child link="grip_attach_1"/>
   <axis xyz="0.0 0.196078 0.980588"/>
+  <dynamics damping="1.0" friction="1.0"/>
 </joint>
 <joint name="slider_left" type="prismatic">
@@ -264,4 +271,5 @@
   <axis xyz="-1.0 0.0 -0.0"/>
   <limit upper="0.0" lower="-0.0455" effort="100" velocity="1.0" acceleration="0.5"/>
+  <dynamics damping="1.0" friction="1.0"/>
 </joint>
 <joint name="slider_right" type="prismatic">
@@ -271,4 +279,5 @@
   <axis xyz="1.0 -0.0 0.0"/>
   <limit upper="0.0" lower="-0.0455" effort="100" velocity="1.0" acceleration="0.5"/>
+  <dynamics damping="1.0" friction="1.0"/>
   <mimic joint="slider_left"/>
 </joint>

Commit message: Restore find command

File: openarm_grip_description/urdf/openarm_grip.urdf (robot description, URDF)
Before this commit: robot openarm_grip, 11 links, 10 joints
Links:
- link J2_v1_1: geometry collision mesh filename=$(find openarm_grip_description)/meshes/J2_v1_1.stl scale=0.001 0.001 0.001; visual mesh filename=$(find openarm_grip_description)/meshes/J2_v1_1.stl scale=0.001 0.001 0.001
- link J3_v1_1: geometry collision mesh filename=$(find openarm_grip_description)/meshes/J3_v1_1.stl scale=0.001 0.001 0.001; visual mesh filename=$(find openarm_grip_description)/meshes/J3_v1_1.stl scale=0.001 0.001 0.001
- link J4_v1_1: geometry collision mesh filename=$(find openarm_grip_description)/meshes/J4_v1_1.stl scale=0.001 0.001 0.001; visual mesh filename=$(find openarm_grip_description)/meshes/J4_v1_1.stl scale=0.001 0.001 0.001
- link J5_v1_1: geometry collision mesh filename=$(find openarm_grip_description)/meshes/J5_v1_1.stl scale=0.001 0.001 0.001; visual mesh filename=$(find openarm_grip_description)/meshes/J5_v1_1.stl scale=0.001 0.001 0.001
- link J6_v1_1: geometry collision mesh filename=$(find openarm_grip_description)/meshes/J6_v1_1.stl scale=0.001 0.001 0.001; visual mesh filename=$(find openarm_grip_description)/meshes/J6_v1_1.stl scale=0.001 0.001 0.001
- link J7_v1_1: geometry collision mesh filename=$(find openarm_grip_description)/meshes/J7_v1_1.stl scale=0.001 0.001 0.001; visual mesh filename=$(find openarm_grip_description)/meshes/J7_v1_1.stl scale=0.001 0.001 0.001
- link base_link: geometry collision mesh filename=$(find openarm_grip_description)/meshes/base_link.stl scale=0.001 0.001 0.001; visual mesh filename=$(find openarm_grip_description)/meshes/base_link.stl scale=0.001 0.001 0.001
- link grip_attach_1: geometry collision mesh filename=$(find openarm_grip_description)/meshes/grip_attach_1.stl scale=0.001 0.001 0.001; visual mesh filename=$(find openarm_grip_description)/meshes/grip_attach_1.stl scale=0.001 0.001 0.001
- link left_jaw_1: geometry collision mesh filename=$(find openarm_grip_description)/meshes/left_jaw_1.stl scale=0.001 0.001 0.001; visual mesh filename=$(find openarm_grip_description)/meshes/left_jaw_1.stl scale=0.001 0.001 0.001
- link right_jaw_1: geometry collision mesh filename=$(find openarm_grip_description)/meshes/right_jaw_1.stl scale=0.001 0.001 0.001; visual mesh filename=$(find openarm_grip_description)/meshes/right_jaw_1.stl scale=0.001 0.001 0.001

File: openarm_grip_description/urdf/openarm_grip.xacro (robot description, xacro)
@@ -1,7 +1,7 @@
 <?xml version="1.0" ?>
 <robot name="openarm_grip" xmlns:xacro="http://www.ros.org/wiki/xacro">
-<xacro:include filename="package://openarm_grip_description/urdf/materials.xacro" />
-<xacro:include filename="package://openarm_grip_description/urdf/openarm_grip.trans" />
-<xacro:include filename="package://openarm_grip_description/urdf/openarm_grip.gazebo" />
+<xacro:include filename="$(find openarm_grip_description)/urdf/materials.xacro" />
+<xacro:include filename="$(find openarm_grip_description)/urdf/openarm_grip.trans" />
+<xacro:include filename="$(find openarm_grip_description)/urdf/openarm_grip.gazebo" />
 <link name="world"/>
 <joint name="world_joint" type="fixed">
@@ -19,5 +19,5 @@
     <origin xyz="0 0 0" rpy="0 0 0"/>
     <geometry>
-      <mesh filename="package://openarm_grip_description/meshes/base_link.stl" scale="0.001 0.001 0.001"/>
+      <mesh filename="$(find openarm_grip_description)/meshes/base_link.stl" scale="0.001 0.001 0.001"/>
     </geometry>
     <material name="silver"/>
@@ -26,5 +26,5 @@
     <origin xyz="0 0 0" rpy="0 0 0"/>
     <geometry>
-      <mesh filename="package://openarm_grip_description/meshes/base_link.stl" scale="0.001 0.001 0.001"/>
+      <mesh filename="$(find openarm_grip_description)/meshes/base_link.stl" scale="0.001 0.001 0.001"/>
     </geometry>
   </collision>
@@ -39,5 +39,5 @@
     <origin xyz="-0.0 -0.0 0.00225" rpy="0 0 0"/>
     <geometry>
-      <mesh filename="package://openarm_grip_description/meshes/J2_v1_1.stl" scale="0.001 0.001 0.001"/>
+      <mesh filename="$(find openarm_grip_description)/meshes/J2_v1_1.stl" scale="0.001 0.001 0.001"/>
     </geometry>
     <material name="silver"/>
@@ -46,5 +46,5 @@
     <origin xyz="-0.0 -0.0 0.00225" rpy="0 0 0"/>
     <geometry>
-      <mesh filename="package://openarm_grip_description/meshes/J2_v1_1.stl" scale="0.001 0.001 0.001"/>
+      <mesh filename="$(find openarm_grip_description)/meshes/J2_v1_1.stl" scale="0.001 0.001 0.001"/>
     </geometry>
   </collision>
@@ -59,5 +59,5 @@
     <origin xyz="-0.02975 0.0 -0.0425" rpy="0 0 0"/>
     <geometry>
-      <mesh filename="package://openarm_grip_description/meshes/J3_v1_1.stl" scale="0.001 0.001 0.001"/>
+      <mesh filename="$(find openarm_grip_description)/meshes/J3_v1_1.stl" scale="0.001 0.001 0.001"/>
     </geometry>
     <material name="silver"/>
@@ -66,5 +66,5 @@
     <origin xyz="-0.02975 0.0 -0.0425" rpy="0 0 0"/>
     <geometry>
-      <mesh filename="package://openarm_grip_description/meshes/J3_v1_1.stl" scale="0.001 0.001 0.001"/>
+      <mesh filename="$(find openarm_grip_description)/meshes/J3_v1_1.stl" scale="0.001 0.001 0.001"/>
     </geometry>
   </collision>
@@ -79,5 +79,5 @@
     <origin xyz="0.0 -0.06041 -0.052607" rpy="0 0 0"/>
     <geometry>
-      <mesh filename="package://openarm_grip_description/meshes/J4_v1_1.stl" scale="0.001 0.001 0.001"/>
+      <mesh filename="$(find openarm_grip_description)/meshes/J4_v1_1.stl" scale="0.001 0.001 0.001"/>
     </geometry>
     <material name="silver"/>
@@ -86,5 +86,5 @@
     <origin xyz="0.0 -0.06041 -0.052607" rpy="0 0 0"/>
     <geometry>
-      <mesh filename="package://openarm_grip_description/meshes/J4_v1_1.stl" scale="0.001 0.001 0.001"/>
+      <mesh filename="$(find openarm_grip_description)/meshes/J4_v1_1.stl" scale="0.001 0.001 0.001"/>
     </geometry>
   </collision>
@@ -99,5 +99,5 @@
     <origin xyz="-0.029755 -0.298846 -0.0925" rpy="0 0 0"/>
     <geometry>
-      <mesh filename="package://openarm_grip_description/meshes/J5_v1_1.stl" scale="0.001 0.001 0.001"/>
+      <mesh filename="$(find openarm_grip_description)/meshes/J5_v1_1.stl" scale="0.001 0.001 0.001"/>
     </geometry>
     <material name="silver"/>
@@ -106,5 +106,5 @@
     <origin xyz="-0.029755 -0.298846 -0.0925" rpy="0 0 0"/>
     <geometry>
-      <mesh filename="package://openarm_grip_description/meshes/J5_v1_1.stl" scale="0.001 0.001 0.001"/>
+      <mesh filename="$(find openarm_grip_description)/meshes/J5_v1_1.stl" scale="0.001 0.001 0.001"/>
     </geometry>
   </collision>
@@ -119,5 +119,5 @@
     <origin xyz="0.0 -0.167496 -0.118765" rpy="0 0 0"/>
     <geometry>
-      <mesh filename="package://openarm_grip_description/meshes/J6_v1_1.stl" scale="0.001 0.001 0.001"/>
+      <mesh filename="$(find openarm_grip_description)/meshes/J6_v1_1.stl" scale="0.001 0.001 0.001"/>
     </geometry>
     <material name="silver"/>
@@ -126,5 +126,5 @@
     <origin xyz="0.0 -0.167496 -0.118765" rpy="0 0 0"/>
     <geometry>
-      <mesh filename="package://openarm_grip_description/meshes/J6_v1_1.stl" scale="0.001 0.001 0.001"/>
+      <mesh filename="$(find openarm_grip_description)/meshes/J6_v1_1.stl" scale="0.001 0.001 0.001"/>
     </geometry>
   </collision>
@@ -139,5 +139,5 @@
     <origin xyz="-0.0355 -0.048796 -0.1425" rpy="0 0 0"/>
     <geometry>
-      <mesh filename="package://openarm_grip_description/meshes/J7_v1_1.stl" scale="0.001 0.001 0.001"/>
+      <mesh filename="$(find openarm_grip_description)/meshes/J7_v1_1.stl" scale="0.001 0.001 0.001"/>
     </geometry>
     <material name="silver"/>
@@ -146,5 +146,5 @@
     <origin xyz="-0.0355 -0.048796 -0.1425" rpy="0 0 0"/>
     <geometry>
-      <mesh filename="package://openarm_grip_description/meshes/J7_v1_1.stl" scale="0.001 0.001 0.001"/>
+      <mesh filename="$(find openarm_grip_description)/meshes/J7_v1_1.stl" scale="0.001 0.001 0.001"/>
     </geometry>
   </collision>
@@ -159,5 +159,5 @@
     <origin xyz="0.0 -0.051826 -0.15765" rpy="0 0 0"/>
     <geometry>
-      <mesh filename="package://openarm_grip_description/meshes/grip_attach_1.stl" scale="0.001 0.001 0.001"/>
+      <mesh filename="$(find openarm_grip_description)/meshes/grip_attach_1.stl" scale="0.001 0.001 0.001"/>
     </geometry>
     <material name="silver"/>
@@ -166,5 +166,5 @@
     <origin xyz="0.0 -0.051826 -0.15765" rpy="0 0 0"/>
     <geometry>
-      <mesh filename="package://openarm_grip_description/meshes/grip_attach_1.stl" scale="0.001 0.001 0.001"/>
+      <mesh filename="$(find openarm_grip_description)/meshes/grip_attach_1.stl" scale="0.001 0.001 0.001"/>
     </geometry>
   </collision>
@@ -179,5 +179,5 @@
     <origin xyz="0.0775 0.069829 -0.169736" rpy="0 0 0"/>
     <geometry>
-      <mesh filename="package://openarm_grip_description/meshes/left_jaw_1.stl" scale="0.001 0.001 0.001"/>
+      <mesh filename="$(find openarm_grip_description)/meshes/left_jaw_1.stl" scale="0.001 0.001 0.001"/>
     </geometry>
     <material name="silver"/>
@@ -186,5 +186,5 @@
     <origin xyz="0.0775 0.069829 -0.169736" rpy="0 0 0"/>
     <geometry>
-      <mesh filename="package://openarm_grip_description/meshes/left_jaw_1.stl" scale="0.001 0.001 0.001"/>
+      <mesh filename="$(find openarm_grip_description)/meshes/left_jaw_1.stl" scale="0.001 0.001 0.001"/>
     </geometry>
   </collision>
@@ -199,5 +199,5 @@
     <origin xyz="-0.0775 0.069829 -0.169736" rpy="0 0 0"/>
     <geometry>
-      <mesh filename="package://openarm_grip_description/meshes/right_jaw_1.stl" scale="0.001 0.001 0.001"/>
+      <mesh filename="$(find openarm_grip_description)/meshes/right_jaw_1.stl" scale="0.001 0.001 0.001"/>
     </geometry>
     <material name="silver"/>
@@ -206,5 +206,5 @@
     <origin xyz="-0.0775 0.069829 -0.169736" rpy="0 0 0"/>
     <geometry>
-      <mesh filename="package://openarm_grip_description/meshes/right_jaw_1.stl" scale="0.001 0.001 0.001"/>
+      <mesh filename="$(find openarm_grip_description)/meshes/right_jaw_1.stl" scale="0.001 0.001 0.001"/>
     </geometry>
   </collision>
