Commit message: Remove all permissions from meshes

File: openarm_grip_description/urdf/openarm_grip.urdf (robot description, URDF)
Before this commit: robot openarm_grip, 11 links, 10 joints
Links:
- link J2_v1_1: geometry collision mesh filename=package://openarm_grip_description/meshes/J2_v1_1.stl scale=0.001 0.001 0.001; visual mesh filename=package://openarm_grip_description/meshes/J2_v1_1.stl scale=0.001 0.001 0.001
- link J3_v1_1: geometry collision mesh filename=package://openarm_grip_description/meshes/J3_v1_1.stl scale=0.001 0.001 0.001; visual mesh filename=package://openarm_grip_description/meshes/J3_v1_1.stl scale=0.001 0.001 0.001
- link J4_v1_1: geometry collision mesh filename=package://openarm_grip_description/meshes/J4_v1_1.stl scale=0.001 0.001 0.001; visual mesh filename=package://openarm_grip_description/meshes/J4_v1_1.stl scale=0.001 0.001 0.001
- link J5_v1_1: geometry collision mesh filename=package://openarm_grip_description/meshes/J5_v1_1.stl scale=0.001 0.001 0.001; visual mesh filename=package://openarm_grip_description/meshes/J5_v1_1.stl scale=0.001 0.001 0.001
- link J6_v1_1: geometry collision mesh filename=package://openarm_grip_description/meshes/J6_v1_1.stl scale=0.001 0.001 0.001; visual mesh filename=package://openarm_grip_description/meshes/J6_v1_1.stl scale=0.001 0.001 0.001
- link J7_v1_1: geometry collision mesh filename=package://openarm_grip_description/meshes/J7_v1_1.stl scale=0.001 0.001 0.001; visual mesh filename=package://openarm_grip_description/meshes/J7_v1_1.stl scale=0.001 0.001 0.001
- link base_link: geometry collision mesh filename=package://openarm_grip_description/meshes/base_link.stl scale=0.001 0.001 0.001; visual mesh filename=package://openarm_grip_description/meshes/base_link.stl scale=0.001 0.001 0.001
- link grip_attach_1: geometry collision mesh filename=package://openarm_grip_description/meshes/grip_attach_1.stl scale=0.001 0.001 0.001; visual mesh filename=package://openarm_grip_description/meshes/grip_attach_1.stl scale=0.001 0.001 0.001
- link left_jaw_1: geometry collision mesh filename=package://openarm_grip_description/meshes/left_jaw_1.stl scale=0.001 0.001 0.001; visual mesh filename=package://openarm_grip_description/meshes/left_jaw_1.stl scale=0.001 0.001 0.001
- link right_jaw_1: geometry collision mesh filename=package://openarm_grip_description/meshes/right_jaw_1.stl scale=0.001 0.001 0.001; visual mesh filename=package://openarm_grip_description/meshes/right_jaw_1.stl scale=0.001 0.001 0.001

File: openarm_grip_description/urdf/openarm_grip.xacro (robot description, xacro)
@@ -19,5 +19,5 @@
     <origin xyz="0 0 0" rpy="0 0 0"/>
     <geometry>
-      <mesh filename="$(find openarm_grip_description)/meshes/base_link.stl" scale="0.001 0.001 0.001"/>
+      <mesh filename="package://openarm_grip_description/meshes/base_link.stl" scale="0.001 0.001 0.001"/>
     </geometry>
     <material name="silver"/>
@@ -26,5 +26,5 @@
     <origin xyz="0 0 0" rpy="0 0 0"/>
     <geometry>
-      <mesh filename="$(find openarm_grip_description)/meshes/base_link.stl" scale="0.001 0.001 0.001"/>
+      <mesh filename="package://openarm_grip_description/meshes/base_link.stl" scale="0.001 0.001 0.001"/>
     </geometry>
   </collision>
@@ -39,5 +39,5 @@
     <origin xyz="-0.0 -0.0 0.00225" rpy="0 0 0"/>
     <geometry>
-      <mesh filename="$(find openarm_grip_description)/meshes/J2_v1_1.stl" scale="0.001 0.001 0.001"/>
+      <mesh filename="package://openarm_grip_description/meshes/J2_v1_1.stl" scale="0.001 0.001 0.001"/>
     </geometry>
     <material name="silver"/>
@@ -46,5 +46,5 @@
     <origin xyz="-0.0 -0.0 0.00225" rpy="0 0 0"/>
     <geometry>
-      <mesh filename="$(find openarm_grip_description)/meshes/J2_v1_1.stl" scale="0.001 0.001 0.001"/>
+      <mesh filename="package://openarm_grip_description/meshes/J2_v1_1.stl" scale="0.001 0.001 0.001"/>
     </geometry>
   </collision>
@@ -59,5 +59,5 @@
     <origin xyz="-0.02975 0.0 -0.0425" rpy="0 0 0"/>
     <geometry>
-      <mesh filename="$(find openarm_grip_description)/meshes/J3_v1_1.stl" scale="0.001 0.001 0.001"/>
+      <mesh filename="package://openarm_grip_description/meshes/J3_v1_1.stl" scale="0.001 0.001 0.001"/>
     </geometry>
     <material name="silver"/>
@@ -66,5 +66,5 @@
     <origin xyz="-0.02975 0.0 -0.0425" rpy="0 0 0"/>
     <geometry>
-      <mesh filename="$(find openarm_grip_description)/meshes/J3_v1_1.stl" scale="0.001 0.001 0.001"/>
+      <mesh filename="package://openarm_grip_description/meshes/J3_v1_1.stl" scale="0.001 0.001 0.001"/>
     </geometry>
   </collision>
@@ -79,5 +79,5 @@
     <origin xyz="0.0 -0.06041 -0.052607" rpy="0 0 0"/>
     <geometry>
-      <mesh filename="$(find openarm_grip_description)/meshes/J4_v1_1.stl" scale="0.001 0.001 0.001"/>
+      <mesh filename="package://openarm_grip_description/meshes/J4_v1_1.stl" scale="0.001 0.001 0.001"/>
     </geometry>
     <material name="silver"/>
@@ -86,5 +86,5 @@
     <origin xyz="0.0 -0.06041 -0.052607" rpy="0 0 0"/>
     <geometry>
-      <mesh filename="$(find openarm_grip_description)/meshes/J4_v1_1.stl" scale="0.001 0.001 0.001"/>
+      <mesh filename="package://openarm_grip_description/meshes/J4_v1_1.stl" scale="0.001 0.001 0.001"/>
     </geometry>
   </collision>
@@ -99,5 +99,5 @@
     <origin xyz="-0.029755 -0.298846 -0.0925" rpy="0 0 0"/>
     <geometry>
-      <mesh filename="$(find openarm_grip_description)/meshes/J5_v1_1.stl" scale="0.001 0.001 0.001"/>
+      <mesh filename="package://openarm_grip_description/meshes/J5_v1_1.stl" scale="0.001 0.001 0.001"/>
     </geometry>
     <material name="silver"/>
@@ -106,5 +106,5 @@
     <origin xyz="-0.029755 -0.298846 -0.0925" rpy="0 0 0"/>
     <geometry>
-      <mesh filename="$(find openarm_grip_description)/meshes/J5_v1_1.stl" scale="0.001 0.001 0.001"/>
+      <mesh filename="package://openarm_grip_description/meshes/J5_v1_1.stl" scale="0.001 0.001 0.001"/>
     </geometry>
   </collision>
@@ -119,5 +119,5 @@
     <origin xyz="0.0 -0.167496 -0.118765" rpy="0 0 0"/>
     <geometry>
-      <mesh filename="$(find openarm_grip_description)/meshes/J6_v1_1.stl" scale="0.001 0.001 0.001"/>
+      <mesh filename="package://openarm_grip_description/meshes/J6_v1_1.stl" scale="0.001 0.001 0.001"/>
     </geometry>
     <material name="silver"/>
@@ -126,5 +126,5 @@
     <origin xyz="0.0 -0.167496 -0.118765" rpy="0 0 0"/>
     <geometry>
-      <mesh filename="$(find openarm_grip_description)/meshes/J6_v1_1.stl" scale="0.001 0.001 0.001"/>
+      <mesh filename="package://openarm_grip_description/meshes/J6_v1_1.stl" scale="0.001 0.001 0.001"/>
     </geometry>
   </collision>
@@ -139,5 +139,5 @@
     <origin xyz="-0.0355 -0.048796 -0.1425" rpy="0 0 0"/>
     <geometry>
-      <mesh filename="$(find openarm_grip_description)/meshes/J7_v1_1.stl" scale="0.001 0.001 0.001"/>
+      <mesh filename="package://openarm_grip_description/meshes/J7_v1_1.stl" scale="0.001 0.001 0.001"/>
     </geometry>
     <material name="silver"/>
@@ -146,5 +146,5 @@
     <origin xyz="-0.0355 -0.048796 -0.1425" rpy="0 0 0"/>
     <geometry>
-      <mesh filename="$(find openarm_grip_description)/meshes/J7_v1_1.stl" scale="0.001 0.001 0.001"/>
+      <mesh filename="package://openarm_grip_description/meshes/J7_v1_1.stl" scale="0.001 0.001 0.001"/>
     </geometry>
   </collision>
@@ -159,5 +159,5 @@
     <origin xyz="0.0 -0.051826 -0.15765" rpy="0 0 0"/>
     <geometry>
-      <mesh filename="$(find openarm_grip_description)/meshes/grip_attach_1.stl" scale="0.001 0.001 0.001"/>
+      <mesh filename="package://openarm_grip_description/meshes/grip_attach_1.stl" scale="0.001 0.001 0.001"/>
     </geometry>
     <material name="silver"/>
@@ -166,5 +166,5 @@
     <origin xyz="0.0 -0.051826 -0.15765" rpy="0 0 0"/>
     <geometry>
-      <mesh filename="$(find openarm_grip_description)/meshes/grip_attach_1.stl" scale="0.001 0.001 0.001"/>
+      <mesh filename="package://openarm_grip_description/meshes/grip_attach_1.stl" scale="0.001 0.001 0.001"/>
     </geometry>
   </collision>
@@ -179,5 +179,5 @@
     <origin xyz="0.0775 0.069829 -0.169736" rpy="0 0 0"/>
     <geometry>
-      <mesh filename="$(find openarm_grip_description)/meshes/left_jaw_1.stl" scale="0.001 0.001 0.001"/>
+      <mesh filename="package://openarm_grip_description/meshes/left_jaw_1.stl" scale="0.001 0.001 0.001"/>
     </geometry>
     <material name="silver"/>
@@ -186,5 +186,5 @@
     <origin xyz="0.0775 0.069829 -0.169736" rpy="0 0 0"/>
     <geometry>
-      <mesh filename="$(find openarm_grip_description)/meshes/left_jaw_1.stl" scale="0.001 0.001 0.001"/>
+      <mesh filename="package://openarm_grip_description/meshes/left_jaw_1.stl" scale="0.001 0.001 0.001"/>
     </geometry>
   </collision>
@@ -199,5 +199,5 @@
     <origin xyz="-0.0775 0.069829 -0.169736" rpy="0 0 0"/>
     <geometry>
-      <mesh filename="$(find openarm_grip_description)/meshes/right_jaw_1.stl" scale="0.001 0.001 0.001"/>
+      <mesh filename="package://openarm_grip_description/meshes/right_jaw_1.stl" scale="0.001 0.001 0.001"/>
     </geometry>
     <material name="silver"/>
@@ -206,5 +206,5 @@
     <origin xyz="-0.0775 0.069829 -0.169736" rpy="0 0 0"/>
     <geometry>
-      <mesh filename="$(find openarm_grip_description)/meshes/right_jaw_1.stl" scale="0.001 0.001 0.001"/>
+      <mesh filename="package://openarm_grip_description/meshes/right_jaw_1.stl" scale="0.001 0.001 0.001"/>
     </geometry>
   </collision>

Commit message: Update rev7 joint type for urdf (continuous -> revolute)

File: openarm_grip_description/urdf/openarm_grip.urdf (robot description, URDF)
Before this commit: robot openarm_grip, 11 links, 10 joints
Joints:
- joint rev7: limit (none) -> lower=-1.5 upper=1.5 effort=100 velocity=1.0; type continuous -> revolute

File: openarm_grip_description/urdf/openarm_grip.xacro (robot description, xacro)
@@ -258,9 +258,10 @@
   <dynamics damping="1.0" friction="1.0"/>
 </joint>
-<joint name="rev7" type="continuous">
+<joint name="rev7" type="revolute">
   <origin xyz="-0.0355 0.00303 0.01515" rpy="0 0 0"/>
   <parent link="J7_v1_1"/>
   <child link="grip_attach_1"/>
   <axis xyz="0.0 0.196078 0.980588"/>
+  <limit upper="0.5" lower="-0.5" effort="100" velocity="1.0" acceleration="0.5"/>
   <dynamics damping="1.0" friction="1.0"/>
 </joint>
