Commit message: Update joint names to be more readable

File: openarm_description/urdf/openarm.urdf (robot description, URDF)
Before this commit: robot openarm, 10 links, 9 joints
Joints:
- removed joint l_J1_v002__to__l_J2_v002
- removed joint l_J2_v002__to__l_J3_v003
- removed joint l_J3_v003__to__l_J4_v002
- removed joint l_J4_v002__to__l_J5_v003
- removed joint l_J5_v003__to__l_J6_v002
- removed joint l_J6_v002__to__l_J7_v002
- removed joint l_J7_v002__to__l_J8_v002
- removed joint l_J8_v002__to__l_left_jaw_v002
- removed joint l_J8_v002__to__l_right_jaw_v002
- added joint gripper_left_jaw: type prismatic, parent l_J8_v002, child l_left_jaw_v002, origin xyz=-0.1071 0.07686 0.0132053 rpy=1.5707963267948268 -0.014066001454925883 0.00875904933451695, axis 0 0 1, limit lower=0.0 upper=0.045 effort=0.0 velocity=0.0
- added joint gripper_right_jaw: type prismatic, parent l_J8_v002, child l_right_jaw_v002, origin xyz=-0.10571 -0.0781373 0.0132053 rpy=1.570796326794885 -0.014066001454926544 0.008759049336297665, axis 0 0 1, limit lower=0.0 upper=0.045 effort=0.0 velocity=0.0, mimic joint=gripper_left_jaw multiplier=-1.0 offset=0.0
- added joint rev1: type revolute, parent l_J1_v002, child l_J2_v002, origin xyz=0.0 0.0 0.05395 rpy=0 0 0, axis 0 0 1, limit lower=-2.356194490192345 upper=2.356194490192345 effort=0.0 velocity=0.0
- added joint rev2: type revolute, parent l_J2_v002, child l_J3_v003, origin xyz=0.0 -0.02975 0.04475 rpy=-1.5707963267948977 1.5707963267948957 0, axis 0 0 1, limit lower=-1.5707963267948966 upper=1.5707963267948966 effort=0.0 velocity=0.0
- added joint rev3: type revolute, parent l_J3_v003, child l_J4_v002, origin xyz=-0.0612477 -0.000536432 0.02975 rpy=1.5707963267949046 0 1.5795545096892487, axis 0 0 1, limit lower=-2.0943951023931953 upper=2.0943951023931953 effort=0.0 velocity=0.0
- added joint rev4: type revolute, parent l_J4_v002, child l_J5_v003, origin xyz=-0.0021149 -0.0318708 -0.241471 rpy=0.7854173400827703 -1.5584104649378014 0.7854173400871975, axis 0 0 1, limit lower=-0.3490658503988659 upper=2.792526803190927 effort=0.0 velocity=0.0
- added joint rev5: type revolute, parent l_J5_v003, child l_J6_v002, origin xyz=-0.133937 0.00188408 -0.0297547 rpy=1.5707963267949707 -0.5569332500522621 1.5567303253381135, axis 0 0 1, limit lower=-2.0943951023931953 upper=2.0943951023931953 effort=0.0 velocity=0.0
- added joint rev6: type revolute, parent l_J6_v002, child l_J7_v002, origin xyz=-0.0187648 -0.0301352 -0.12105 rpy=-1.5707963268025373 -1.5567303253381704 -0.5569332500438752, axis 0 0 1, limit lower=-1.5707963267948966 upper=1.5707963267948966 effort=0.0 velocity=0.0
- added joint rev7: type revolute, parent l_J7_v002, child l_J8_v002, origin xyz=-0.000217313 -0.0154485 0.0355 rpy=-1.570796326795002 -0.008759049335348993 -0.014066001454933549, axis 0 0 1, limit lower=-0.9599310885968813 upper=0.9599310885968813 effort=0.0 velocity=0.0
