Commit message: Implement openarm ros2_control support with openarm_hardware and openarm_bringup (#2)
- openarm_bringup: ros2_control bringup
- openarm_hardware: hardware interface for ros2_control

File: openarm_description/urdf/openarm.ros2_control.xacro (robot description, xacro)
@@ -1,82 +1,93 @@
 <?xml version="1.0"?>
 <robot xmlns:xacro="http://www.ros.org/wiki/xacro">
-    <xacro:macro name="openarm_grip_ros2_control" params="name initial_positions_file">
+    <xacro:macro name="openarm_ros2_control" params="name initial_positions_file prefix:=''">
         <xacro:property name="initial_positions" value="${xacro.load_yaml(initial_positions_file)['initial_positions']}"/>
-        <ros2_control name="${name}" type="system">
+        <ros2_control name="${prefix}${name}" type="system">
             <hardware>
                 <!-- By default, set up controllers for simulation. This won't work on real hardware -->
                 <plugin>mock_components/GenericSystem</plugin>
+                <plugin>openarm_hardware/OpenArmHW</plugin>
             </hardware>
-            <joint name="rev1">
+            <joint name="${prefix}rev1">
                 <command_interface name="position"/>
                 <command_interface name="velocity"/>
+                <command_interface name="effort"/>
                 <state_interface name="position">
                   <param name="initial_value">${initial_positions['rev1']}</param>
                 </state_interface>
                 <state_interface name="velocity"/>
+                <state_interface name="effort"/>
             </joint>
-            <joint name="rev2">
+            <joint name="${prefix}rev2">
                 <command_interface name="position"/>
                 <command_interface name="velocity"/>
+                <command_interface name="effort"/>
                 <state_interface name="position">
                   <param name="initial_value">${initial_positions['rev2']}</param>
                 </state_interface>
                 <state_interface name="velocity"/>
+                <state_interface name="effort"/>
             </joint>
-            <joint name="rev3">
+            <joint name="${prefix}rev3">
                 <command_interface name="position"/>
                 <command_interface name="velocity"/>
+                <command_interface name="effort"/>
                 <state_interface name="position">
                   <param name="initial_value">${initial_positions['rev3']}</param>
                 </state_interface>
                 <state_interface name="velocity"/>
+                <state_interface name="effort"/>
             </joint>
-            <joint name="rev4">
+            <joint name="${prefix}rev4">
                 <command_interface name="position"/>
                 <command_interface name="velocity"/>
+                <command_interface name="effort"/>
                 <state_interface name="position">
                   <param name="initial_value">${initial_positions['rev4']}</param>
                 </state_interface>
                 <state_interface name="velocity"/>
+                <state_interface name="effort"/>
             </joint>
-            <joint name="rev5">
+            <joint name="${prefix}rev5">
                 <command_interface name="position"/>
                 <command_interface name="velocity"/>
+                <command_interface name="effort"/>
                 <state_interface name="position">
                   <param name="initial_value">${initial_positions['rev5']}</param>
                 </state_interface>
                 <state_interface name="velocity"/>
+                <state_interface name="effort"/>
             </joint>
-            <joint name="rev6">
+            <joint name="${prefix}rev6">
                 <command_interface name="position"/>
                 <command_interface name="velocity"/>
+                <command_interface name="effort"/>
                 <state_interface name="position">
                   <param name="initial_value">${initial_positions['rev6']}</param>
                 </state_interface>
                 <state_interface name="velocity"/>
+                <state_interface name="effort"/>
             </joint>
-            <joint name="rev7">
+            <joint name="${prefix}rev7">
                 <command_interface name="position"/>
                 <command_interface name="velocity"/>
+                <command_interface name="effort"/>
                 <state_interface name="position">
                   <param name="initial_value">${initial_positions['rev7']}</param>
                 </state_interface>
                 <state_interface name="velocity"/>
+                <state_interface name="effort"/>
             </joint>
-            <joint name="slider_left">
+            <joint name="${prefix}left_pris1">
                 <command_interface name="position"/>
-                <command_interface name="velocity"/>
                 <state_interface name="position">
-                  <param name="initial_value">${initial_positions['slider_left']}</param>
+                  <param name="initial_value">${initial_positions['left_pris1']}</param>
                 </state_interface>
                 <state_interface name="velocity"/>
             </joint>
-            <joint name="slider_right">
-                <command_interface name="position"/>
-                <command_interface name="velocity"/>
+            <joint name="${prefix}right_pris2">
                 <state_interface name="position">
-                  <param name="initial_value">${initial_positions['slider_right']}</param>
+                  <param name="initial_value">${initial_positions['left_pris1']}</param>
                 </state_interface>
-                <state_interface name="velocity"/>
             </joint>
         </ros2_control>

File: openarm_description/urdf/openarm.xacro (robot description, xacro)
@@ -10,4 +10,8 @@
         <xacro:property name="reflect" value="${1 if side=='right' else -1}"/>
         <xacro:property name="rotate" value="${0 if side=='right' else pi}"/>
+        <xacro:include filename="openarm_sensors.urdf.xacro"/>
+        <xacro:arg name="initial_positions_file" default="initial_positions.yaml" />
+        <xacro:include filename="openarm.ros2_control.xacro" />
+        <xacro:openarm_ros2_control name="OpenArmHW" prefix="${prefix}" initial_positions_file="$(arg initial_positions_file)"/>
         <link name="${prefix}link1">
             <visual>
