Commit message: Resolve merge conflict

File: openarm_description/urdf/openarm.xacro (robot description, xacro)
@@ -181,4 +181,5 @@
             </inertial>
         </link>
+        <link name="${prefix}gripper_center"/>
         <link name="${prefix}link_left_jaw">
             <visual>
@@ -285,4 +286,9 @@
             <mimic joint="${prefix}left_pris1" multiplier="-1.0" offset="0.0"/>
         </joint>
+        <joint name="${prefix}virtual_gripper_center" type="fixed">
+            <parent link="${prefix}link8"/>
+            <child link="${prefix}gripper_center"/>
+            <origin rpy="0 0 0" xyz="-0.13 0.00 0.0132053"/>
+        </joint>
     </xacro:macro>
 </robot>

Commit message: Correct URDF to true joint limits + Add and update documentation (#6)
* Rename openarm_bimanual_teleop to openarm_bimanual_bringup

* Update package descriptions

* Add quickstart link

* Add note to source overlay

* Add test installation step

* Add poses and update default rviz config

* Fix rev1 to match hardware

* Align rev3 with hardware joint limits

* Match hardware joint limits

* Complete with more poses

* Update README.md with moveit2 video

* Add new READMEs in openarm_bringup and openarm_bimanual_moveit_config

* Add octomap note

File: openarm_description/urdf/openarm.xacro (robot description, xacro)
@@ -227,5 +227,5 @@
             <origin rpy="0 0 0" xyz="0.0 0.0 0.05325"/>
             <axis xyz="0 0 1"/>
-            <limit effort="0.0" lower="-2.0943951023931953" upper="2.0943951023931953" velocity="0.0"/>
+            <limit effort="0.0" lower="${-pi/4.0 if side=='right' and zero_pos=='arm' else -2.0943951023931953}" upper="${pi/4.0 if side=='left' and zero_pos=='arm' else 2.0943951023931953}" velocity="0.0"/>
         </joint>
         <joint name="${prefix}rev2" type="revolute">
@@ -234,5 +234,5 @@
             <origin rpy="-1.5707963267948968 ${pi/2 if zero_pos=='up' else 0.0} 0.0" xyz="0.0 -0.02975 0.04475"/>
             <axis xyz="0 0 1"/>
-            <limit effort="0.0" lower="${-pi/2.0 if zero_pos=='up' else 0}" upper="${pi/2 if zero_pos=='up' else pi}" velocity="0.0"/>
+            <limit effort="0.0" lower="${-pi/2.0 if zero_pos=='up' else -pi/18.0}" upper="${pi/2 if zero_pos=='up' else pi * 17.0 / 18.0}" velocity="0.0"/>
         </joint>
         <joint name="${prefix}rev3" type="revolute">
@@ -241,5 +241,5 @@
             <origin rpy="-1.5707963267949054 ${rotate} -1.562038143900564" xyz="-0.0612477 -0.000536432 0.02975"/>
             <axis xyz="0 0 -1"/>
-            <limit effort="0.0" lower="${-0.52359 if side=='right' else -3.66519}" upper="${3.66519 if side=='right' else 0.52359}" velocity="0.0"/>
+            <limit effort="0.0" lower="${-pi * 2.0 / 3.0}" upper="${pi * 2.0 / 3.0}" velocity="0.0"/>
         </joint>
         <joint name="${prefix}rev4" type="revolute">
@@ -248,5 +248,5 @@
             <origin rpy="-0.20701608758495998 -1.5707963267948566 -2.937419385117548" xyz="0.0297547 0.0 -0.24175"/>
             <axis xyz="0 0 1"/>
-            <limit effort="0.0" lower="-0.3490658503988659" upper="2.792526803190927" velocity="0.0"/>
+            <limit effort="0.0" lower="0" upper="${pi * 5.0 / 6.0}" velocity="0.0"/>
         </joint>
         <joint name="${prefix}rev5" type="revolute">
@@ -255,5 +255,5 @@
             <origin rpy="1.5707963267948473 -0.5569332500492129 1.556730325338251" xyz="-0.133937 0.00188408 -0.0297547"/>
             <axis xyz="0 0 -1"/>
-            <limit effort="0.0" lower="-2.0943951023931953" upper="2.0943951023931953" velocity="0.0"/>
+            <limit effort="0.0" lower="${-pi * 2.0 / 3.0}" upper="${pi * 2.0 / 3.0}" velocity="0.0"/>
         </joint>
         <joint name="${prefix}rev6" type="revolute">
@@ -262,5 +262,5 @@
             <origin rpy="-1.5707963268024898 -1.5567303253382425 -0.5569332500461536" xyz="-0.0187648 -0.0301352 -0.12105"/>
             <axis xyz="0 0 ${reflect}"/>
-            <limit effort="0.0" lower="-1.5707963267948966" upper="1.5707963267948966" velocity="0.0"/>
+            <limit effort="0.0" lower="${-pi / 2.0}" upper="${pi / 2.0}" velocity="0.0"/>
         </joint>
         <joint name="${prefix}rev7" type="revolute">
@@ -269,5 +269,5 @@
             <origin rpy="-1.5707963267950005 -0.00875904933536772 -0.014066001454933467" xyz="-0.000217313 -0.0154485 0.0355"/>
             <axis xyz="0 0 -1"/>
-            <limit effort="0.0" lower="-0.9599310885968813" upper="0.9599310885968813" velocity="0.0"/>
+            <limit effort="0.0" lower="${-pi * 11.0 / 36.0}" upper="${pi * 11.0 / 36.0}" velocity="0.0"/>
         </joint>
         <joint name="${prefix}left_pris1" type="prismatic">
