Commit message: Add left and right arms

File: openarm_two_arms/urdf/openarm_left.urdf (robot description, URDF)
Before this commit: robot openarm_two_arms, 0 links, 9 joints
Links:
- added link l_J2_v003, mass 0.16257504134917358; collision box size=0.059000000014901216 0.08200000000000003 0.0742471498637348; visual mesh filename=package://openarm_two_arms/meshes/full_upper_j2v2_gscnlc.dae
- added link l_J3_v004, mass 0.42038984024444975; collision box size=0.0898910738785183 0.06999999999999985 0.05902136986134156; visual mesh filename=package://openarm_two_arms/meshes/full_upper_j3v005_2vn1gz.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
- added link l_J4_v003, mass 0.8196402299327217; collision box size=0.27584679830769426 0.08211367789676165 0.07185639591248483; visual mesh filename=package://openarm_two_arms/meshes/full_upper_j4v2_tzaxwp.dae
- added link l_J5_v004, mass 0.40867482543516; collision box size=0.1676296341613413 0.06430555048399128 0.08257859967140607; visual mesh filename=package://openarm_two_arms/meshes/full_upper_j5v005_didwyo.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
- added link l_J6_Left_v004, mass 0.34433331594607314; collision box size=0.1311435300470597 0.059534783253118076 0.08817198167731641; visual mesh filename=package://openarm_two_arms/meshes/full_upper_j6_leftv005_f8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
- added link l_J7_Left_v004, mass 0.2782996911629702; collision box size=0.05859778949354245 0.04469786051400639 0.08267618289454949; visual mesh filename=package://openarm_two_arms/meshes/full_upper_j7_leftv005_8o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
- added link l_J8_v003, mass 0.3126145274380216; collision box size=0.1302624002952524 0.052571684700854236 0.1601213740691585; visual mesh filename=package://openarm_two_arms/meshes/full_upper_j8v004_upij9o.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
- added link l_base_link001, mass 0.5769283920617254; collision box size=0.11 0.073 0.0592; visual mesh filename=package://openarm_two_arms/meshes/full_upper_base_link_int1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
- added link l_left_jaw_v004, mass 0.04297897856394934; collision mesh filename=package://openarm_two_arms/meshes/full_upper_col_left_jaw_v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; visual mesh filename=package://openarm_two_arms/meshes/full_upper_left_jawv003_9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
- added link l_right_jaw_v004, mass 0.042981665301134495; collision mesh filename=package://openarm_two_arms/meshes/full_upper_col_right_jaw_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; visual mesh filename=package://openarm_two_arms/meshes/full_upper_right_jawv003_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

File: openarm_two_arms/urdf/openarm_right.urdf (robot description, URDF)
Before this commit: robot openarm_two_arms, 20 links, 9 joints
Links:
- removed link l_J2_v003
- removed link l_J3_v004
- removed link l_J4_v003
- removed link l_J5_v004
- removed link l_J6_Left_v004
- removed link l_J7_Left_v004
- removed link l_J8_v003
- removed link l_base_link001
- removed link l_left_jaw_v004
- removed link l_right_jaw_v004
