Commit message: Define xacro shortcuts to start and decouple left and right arms from torso

File: openarm_two_arms/urdf/openarm_two_arms.urdf (robot description, URDF)
Before this commit: robot openarm_two_arms, 21 links, 20 joints
Links:
- removed link l_pedestal_02_urdf_v002
- added link pedestal_link, mass 4.850309883435878; collision box size=0.18 0.06 0.978000000000004; visual mesh filename=package://openarm_two_arms/meshes/full_upper_pedestal_02_ur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
Joints:
- joint left_fix1: parent l_pedestal_02_urdf_v002 -> pedestal_link
- joint right_fix1: parent l_pedestal_02_urdf_v002 -> pedestal_link

Commit message: Generate updated urdf

File: openarm_two_arms/urdf/openarm_two_arms.urdf (robot description, URDF)
Before this commit: robot openarm_two_arms, 22 links, 21 joints
Joints:
- removed joint left_fix1
- removed joint right_fix1
- added joint left_fixed1: type fixed, parent pedestal_link, child right_link1, origin xyz=-0.09 0.0 0.893 rpy=6.160245846096606 -1.5707963267948268 0.12293946108298068
- added joint right_fixed1: type fixed, parent pedestal_link, child left_link1, origin xyz=0.09 0.0 0.893 rpy=3.0144791747751833 -1.5707963267948324 0.12689401604101067
