Commit message: Switch default to right

File: openarm_two_arms/urdf/openarm_left.urdf (robot description, URDF)
Before this commit: robot openarm_two_arms, 10 links, 9 joints
Links:
- removed link l_base_link001
- added link left_link1, mass 0.5769283920617254; collision box size=0.11 0.073 0.0592; visual mesh filename=package://openarm_two_arms/meshes/full_upper_base_link_int1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
Joints:
- joint left_rev1: parent l_base_link001 -> left_link1

File: openarm_two_arms/urdf/openarm_two_arms.urdf.xacro (robot description, xacro)
@@ -4,6 +4,6 @@
   <xacro:include filename="openarm.xacro"/>
   <xacro:include filename="openarm_two_arms_pedestal.urdf"/>
-  <xacro:openarm prefix="left_" side="left"/>
-  <xacro:include filename="openarm_right.urdf"/>
+  <xacro:openarm prefix="right_" side="right"/>
+  <xacro:include filename="openarm_left.urdf"/>
   <joint name="dummy_joint" type="fixed">
     <parent link="world"/>
@@ -13,5 +13,5 @@
   <joint name="right_fix1" type="fixed">
     <parent link="pedestal_link"/>
-    <child link="l_J1_v002"/>
+    <child link="right_link1"/>
     <origin rpy="3.0144791747751833 -1.5707963267948324 0.12689401604101067" xyz="0.09 0.0 0.893"/>
   </joint>

Commit message: Checkpoint: up to link3

File: openarm_two_arms/urdf/openarm.xacro (robot description, xacro)
@@ -3,12 +3,12 @@
     <xacro:property name="side" value="right"/>
     <xacro:property name="prefix" value=""/>
-    <xacro:property name="pi" value="3.1415926535897927"/>
+    <!-- <xacro:property name="pi" value="3.1415926535897927"/> -->
     <!-- <xacro:property name="zero_pos" value="vertical"/> -->
     <xacro:macro name="openarm" params="side prefix">
-        <xacro:property name="reflect" value ="${(arm_side=='right') ? '1' : '-1'}"/>
+        <xacro:property name="reflect" value ="${ 1 if side=='right' else -1}"/>
         <link name="${prefix}link1">
             <visual>
                 <!--J1 v002/Part__Feature001.-->
-                <origin rpy="0 0 0" xyz="0.0 0.0 -0.0007"/>
+                <origin rpy="${0 if side=='right' else pi} 0 0" xyz="0.0 0.0 ${reflect*0.0007}"/>
                 <geometry>
                     <mesh filename="package://openarm_two_arms/meshes/full_upper_j1v1_fj2ul1.dae"/>
@@ -17,5 +17,5 @@
             <collision>
                 <!--bound_obj__right_link1__col_J1_v1__BoundBox/col_J1_v1__BoundBox.-->
-                <origin rpy="0 0 0" xyz="0.0 0.0 0.0289"/>
+                <origin rpy="${0 if side=='right' else pi} 0 0" xyz="0.0 0.0 ${reflect*0.0289}"/>
                 <geometry>
                     <box size="0.11 0.073 0.0592"/>
@@ -24,5 +24,5 @@
             <inertial>
                 <mass value="0.5769283920617254"/>
-                <origin rpy="0 0 0" xyz="0.0 2.52845e-05 0.0229621"/>
+                <origin rpy="${0 if side=='right' else pi} 0 0" xyz="0.0 2.52845e-05 0.0229621"/>
                 <inertia ixx="0.00034035167574060775" ixy="-2.623557985991217e-18" ixz="-6.093726095527621e-18" iyy="0.0004300058300010205" iyz="-5.09829482074806e-07" izz="0.0004802171432001996"/>
             </inertial>

Commit message: Correct first joint of left arm

File: openarm_two_arms/urdf/openarm.xacro (robot description, xacro)
@@ -10,5 +10,5 @@
             <visual>
                 <!--J1 v002/Part__Feature001.-->
-                <origin rpy="${0 if side=='right' else pi} 0 0" xyz="0.0 0.0 ${reflect*0.0007}"/>
+                <origin rpy="${0 if side=='right' else pi} 0 0" xyz="0.0 0.0 ${reflect*-0.0007}"/>
                 <geometry>
                     <mesh filename="package://openarm_two_arms/meshes/full_upper_j1v1_fj2ul1.dae"/>
@@ -24,5 +24,5 @@
             <inertial>
                 <mass value="0.5769283920617254"/>
-                <origin rpy="${0 if side=='right' else pi} 0 0" xyz="0.0 2.52845e-05 0.0229621"/>
+                <origin rpy="${0 if side=='right' else pi} 0 0" xyz="0.0 ${reflect*2.52845e-05} ${reflect*0.0229621}"/>
                 <inertia ixx="0.00034035167574060775" ixy="-2.623557985991217e-18" ixz="-6.093726095527621e-18" iyy="0.0004300058300010205" iyz="-5.09829482074806e-07" izz="0.0004802171432001996"/>
             </inertial>
@@ -31,5 +31,5 @@
             <visual>
                 <!--J2 v002/Part__Feature002.-->
-                <origin rpy="0 0 0" xyz="0.0 0.0 -0.05395"/>
+                <origin rpy="${0 if side=='right' else pi} 0 0" xyz="0.0 0.0 ${reflect*-0.05395}"/>
                 <geometry>
                     <mesh filename="package://openarm_two_arms/meshes/full_upper_j2v1_xzm1cu.dae"/>
@@ -38,5 +38,5 @@
             <collision>
                 <!--bound_obj__right_link2__col_J2_v1__BoundBox/col_J2_v1__BoundBox.-->
-                <origin rpy="0 0 0" xyz="0.0 0.0 0.0371236"/>
+                <origin rpy="${0 if side=='right' else pi} 0 0" xyz="0.0 0.0 ${reflect*0.0371236}"/>
                 <geometry>
                     <box size="0.0590000000149012 0.08200000000000002 0.0742471498637348"/>
@@ -45,6 +45,6 @@
             <inertial>
                 <mass value="0.16257504134917358"/>
-                <origin rpy="0 0 0" xyz="-0.000225878 -0.00183836 0.0278368"/>
-                <inertia ixx="0.00023903110213294374" ixy="-7.551692921096027e-08" ixz="-1.1282723362433474e-06" iyy="0.00010490798314778774" iyz="5.9079627839725245e-06" izz="0.00019737368685935776"/>
+                <origin rpy="0 0 0" xyz="${reflect*-0.000225878} ${reflect*-0.00183836} 0.0278368"/>
+                <inertia ixx="0.00023903110213294374" ixy="-7.551692921096027e-08" ixz="${reflect*-1.1282723362433474e-06}" iyy="0.00010490798314778774" iyz="${reflect*5.9079627839725245e-06}" izz="0.00019737368685935776"/>
             </inertial>
         </link>
@@ -52,5 +52,5 @@
             <visual>
                 <!--J3 v003/Part__Feature003.-->
-                <origin rpy="1.570796326794897 0 0" xyz="0.0 0.0987 0.02975"/>
+                <origin rpy="1.570796326794897 0 0" xyz="0.0 0.0987 ${reflect*0.02975}"/>
                 <geometry>
                     <mesh filename="package://openarm_two_arms/meshes/full_upper_j3v2_5nirfo.dae"/>
@@ -66,6 +66,6 @@
             <inertial>
                 <mass value="0.4201676469910031"/>
-                <origin rpy="1.5707963267948968 0 0" xyz="-0.00688022 0.0 0.0282752"/>
-                <inertia ixx="0.00020256001126230057" ixy="6.004247875311213e-06" ixz="1.3304903057525575e-06" iyy="0.0002970624991387495" iyz="5.980157765704868e-07" izz="0.00032889994351244413"/>
+                <origin rpy="1.5707963267948968 0 0" xyz="${reflect*-0.00688022} 0.0 0.0282752"/>
+                <inertia ixx="0.00020256001126230057" ixy="6.004247875311213e-06" ixz="${reflect*1.3304903057525575e-06}" iyy="0.0002970624991387495" iyz="${reflect*5.980157765704868e-07}" izz="0.00032889994351244413"/>
             </inertial>
         </link>
@@ -112,5 +112,5 @@
             </inertial>
         </link>
-        <link name="l_J6_right_wrist">
+        <link name="${prefix}link6_right_wrist">
             <visual>
                 <!--J6 right_wrist/Part__Feature006.-->
@@ -175,5 +175,5 @@
             </inertial>
         </link>
-        <link name="l_left_jaw_v002">
+        <link name="${prefix}link_left_jaw">
             <visual>
                 <!--left_jaw v002/Part__Feature009.-->
@@ -196,5 +196,5 @@
             </inertial>
         </link>
-        <link name="l_right_jaw_v002">
+        <link name="${prefix}link_right_jaw">
             <visual>
                 <!--right_jaw v002/Part__Feature010.-->
@@ -217,26 +217,26 @@
             </inertial>
         </link>
-        <joint name="right_rev1" type="revolute">
+        <joint name="${prefix}rev1" type="revolute">
             <parent link="${prefix}link1"/>
             <child link="${prefix}link2"/>
-            <origin rpy="0 0 0" xyz="0.0 0.0 0.05325"/>
+            <origin rpy="${0 if side=='right' else -pi} ${0 if side=='right' else -pi} 0" xyz="0.0 0.0 ${reflect*0.05325}"/>
             <axis xyz="0 0 1"/>
             <limit effort="0.0" lower="-2.0943951023931953" upper="2.0943951023931953" velocity="0.0"/>
         </joint>
-        <joint name="right_rev2" type="revolute">
+        <joint name="${prefix}rev2" type="revolute">
             <parent link="${prefix}link2"/>
             <child link="${prefix}link3"/>
-            <origin rpy="-1.5707963267948968 0 0" xyz="0.0 -0.02975 0.04475"/>
-            <axis xyz="0 0 1"/>
-            <limit effort="0.0" lower="0.0" upper="3.141592653589793" velocity="0.0"/>
-        </joint>
-        <joint name="right_rev3" type="revolute">
+            <origin rpy="-1.5707963267948968 0 0" xyz="0.0 ${reflect*-0.02975} 0.04475"/>
+            <axis xyz="0 0 1"/>
+            <limit effort="0.0" lower="${0.0 if side=='right' else -pi}" upper="${pi if side=='right' else 0.0}" velocity="0.0"/>
+        </joint>
+        <joint name="${prefix}rev3" type="revolute">
             <parent link="${prefix}link3"/>
             <child link="${prefix}link4"/>
-            <origin rpy="-1.5707963267949054 0 -1.562038143900564" xyz="-0.0612477 -0.000536432 0.02975"/>
+            <origin rpy="${reflect*-1.5707963267949054} 0 ${reflect*-1.562038143900564}" xyz="${reflect*-0.0612477} -0.000536432 ${reflect*0.02975}"/>
             <axis xyz="0 0 1"/>
             <limit effort="0.0" lower="-3.6651914291880923" upper="0.5235987755982988" velocity="0.0"/>
         </joint>
-        <joint name="right_rev4" type="revolute">
+        <joint name="${prefix}rev4" type="revolute">
             <parent link="${prefix}link4"/>
             <child link="${prefix}link5"/>
@@ -245,13 +245,13 @@
             <limit effort="0.0" lower="-0.3490658503988659" upper="2.792526803190927" velocity="0.0"/>
         </joint>
-        <joint name="right_rev5" type="revolute">
+        <joint name="${prefix}rev5" type="revolute">
             <parent link="${prefix}link5"/>
-            <child link="l_J6_right_wrist"/>
+            <child link="${prefix}link6_right_wrist"/>
             <origin rpy="1.5707963267948473 -0.5569332500492129 1.556730325338251" xyz="-0.133937 0.00188408 -0.0297547"/>
             <axis xyz="0 0 1"/>
             <limit effort="0.0" lower="-2.0943951023931953" upper="2.0943951023931953" velocity="0.0"/>
         </joint>
-        <joint name="right_rev6" type="revolute">
-            <parent link="l_J6_right_wrist"/>
+        <joint name="${prefix}rev6" type="revolute">
+            <parent link="${prefix}link6_right_wrist"/>
             <child link="${prefix}link7"/>
             <origin rpy="-1.5707963268024898 -1.5567303253382425 -0.5569332500461536" xyz="-0.0187648 -0.0301352 -0.12105"/>
@@ -259,5 +259,5 @@
             <limit effort="0.0" lower="-1.5707963267948966" upper="1.5707963267948966" velocity="0.0"/>
         </joint>
-        <joint name="right_rev7" type="revolute">
+        <joint name="${prefix}rev7" type="revolute">
             <parent link="${prefix}link7"/>
             <child link="${prefix}link8"/>
@@ -266,18 +266,18 @@
             <limit effort="0.0" lower="-0.9599310885968813" upper="0.9599310885968813" velocity="0.0"/>
         </joint>
-        <joint name="right_left_pris1" type="prismatic">
+        <joint name="${prefix}left_pris1" type="prismatic">
             <parent link="${prefix}link8"/>
-            <child link="l_left_jaw_v002"/>
+            <child link="${prefix}link_left_jaw"/>
             <origin rpy="1.570796326795101 -0.014066001454929162 0.00875904933542146" xyz="-0.1071 0.0768568 0.0132053"/>
             <axis xyz="0 0 1"/>
             <limit effort="0.0" lower="0.0" upper="0.045" velocity="0.0"/>
         </joint>
-        <joint name="right_right_pris2" type="prismatic">
+        <joint name="${prefix}right_pris2" type="prismatic">
             <parent link="${prefix}link8"/>
-            <child link="l_right_jaw_v002"/>
+            <child link="${prefix}link_right_jaw"/>
             <origin rpy="1.570796326794883 -0.014066001454927403 0.008759049336290027" xyz="-0.10571 -0.0781373 0.0132053"/>
             <axis xyz="0 0 1"/>
             <limit effort="0.0" lower="0.0" upper="0.045" velocity="0.0"/>
-            <mimic joint="right_left_pris1" multiplier="-1.0" offset="0.0"/>
+            <mimic joint="${prefix}left_pris1" multiplier="-1.0" offset="0.0"/>
         </joint>
     </xacro:macro>

File: openarm_two_arms/urdf/openarm_two_arms.urdf.xacro (robot description, xacro)
@@ -5,5 +5,6 @@
   <xacro:include filename="openarm_two_arms_pedestal.urdf"/>
   <xacro:openarm prefix="right_" side="right"/>
-  <xacro:include filename="openarm_left.urdf"/>
+  <xacro:openarm prefix="left_" side="left"/>
+  <!-- <xacro:include filename="openarm_left.urdf"/> -->
   <joint name="dummy_joint" type="fixed">
     <parent link="world"/>

Commit message: Checkpoint to add up to rev 6, link 4

File: openarm_two_arms/urdf/openarm.xacro (robot description, xacro)
@@ -241,12 +241,12 @@
             <parent link="${prefix}link4"/>
             <child link="${prefix}link5"/>
-            <origin rpy="-0.20701608758495998 -1.5707963267948566 -2.937419385117548" xyz="0.0297547 0.0 -0.24175"/>
-            <axis xyz="0 0 1"/>
-            <limit effort="0.0" lower="-0.3490658503988659" upper="2.792526803190927" velocity="0.0"/>
+            <origin rpy="${-0.20701608758495998 if side=='right' else -3.0383286058327292} -1.5707963267948566 ${-2.937419385117548 if side=='right' else 3.038328605832587}" xyz="0.0297547 0.0 ${reflect*-0.24175}"/>
+            <axis xyz="0 0 1"/>
+            <limit effort="0.0" lower="${-0.3490658503988659 if side=='right' else -2.792526803190927}" upper="${2.792526803190927 if side=='right' else 0.3490658503988659}" velocity="0.0"/>
         </joint>
         <joint name="${prefix}rev5" type="revolute">
             <parent link="${prefix}link5"/>
             <child link="${prefix}link6_right_wrist"/>
-            <origin rpy="1.5707963267948473 -0.5569332500492129 1.556730325338251" xyz="-0.133937 0.00188408 -0.0297547"/>
+            <origin rpy="${reflect*1.5707963267948473} ${reflect*-0.5569332500492129} 1.556730325338251" xyz="${reflect*-0.133937} 0.00188408 ${reflect*-0.0297547}"/>
             <axis xyz="0 0 1"/>
             <limit effort="0.0" lower="-2.0943951023931953" upper="2.0943951023931953" velocity="0.0"/>
@@ -255,5 +255,5 @@
             <parent link="${prefix}link6_right_wrist"/>
             <child link="${prefix}link7"/>
-            <origin rpy="-1.5707963268024898 -1.5567303253382425 -0.5569332500461536" xyz="-0.0187648 -0.0301352 -0.12105"/>
+            <origin rpy="${reflect*-1.5707963268024898} -1.5567303253382425 -0.5569332500461536" xyz="${reflect*-0.0187648} ${reflect*-0.0301352} ${reflect*-0.12105}"/>
             <axis xyz="0 0 1"/>
             <limit effort="0.0" lower="-1.5707963267948966" upper="1.5707963267948966" velocity="0.0"/>

Commit message: Link 5 checkpoint

File: openarm_two_arms/urdf/openarm.xacro (robot description, xacro)
@@ -94,5 +94,5 @@
             <visual>
                 <!--J5 v003/Part__Feature005.-->
-                <origin rpy="0 -0.008758182894317394 0" xyz="0.303864 0.0 -0.128451"/>
+                <origin rpy="0 ${reflect*-0.008758182894317394} 0" xyz="${reflect*0.303864} 0.0 ${-0.128451 if side=='right' else -0.0689415"/>
                 <geometry>
                     <mesh filename="package://openarm_two_arms/meshes/full_upper_j5v2_ckk9an.dae"/>
@@ -101,5 +101,5 @@
             <collision>
                 <!--bound_obj__right_link5__col_J5_v2__BoundBox/col_J5_v2__BoundBox.-->
-                <origin rpy="0 -0.008758182894316818 0" xyz="-0.0542814 0.00265291 -0.0302022"/>
+                <origin rpy="0 ${reflect*-0.008758182894316818} 0" xyz="${reflect*-0.0542814} 0.00265291 ${reflect*-0.0302022}"/>
                 <geometry>
                     <box size="0.16827213220625828 0.06430555048399171 0.08257859967140947"/>
@@ -108,6 +108,6 @@
             <inertial>
                 <mass value="0.4086748254352304"/>
-                <origin rpy="0 -0.008758182894316905 0" xyz="-0.0831891 0.00251789 -0.0290107"/>
-                <inertia ixx="0.00031417157425298747" ixy="-1.1391566029536723e-05" ixz="-1.883474090056124e-05" iyy="0.001221711435313989" iyz="1.46725418421127e-06" izz="0.0010755135067660488"/>
+                <origin rpy="0 ${reflect*-0.008758182894316905} 0" xyz="${reflect*-0.0831891} 0.00251789 ${reflect*-0.0290107}"/>
+                <inertia ixx="0.00031417157425298747" ixy="${reflect*-1.1391566029536723e-05}" ixz="${reflect*-1.883474090056124e-05}" iyy="0.001221711435313989" iyz="${reflect*1.46725418421127e-06}" izz="0.0010755135067660488"/>
             </inertial>
         </link>
