Commit message: Add left wrist

File: openarm_two_arms/urdf/openarm.xacro (robot description, xacro)
@@ -113,10 +113,10 @@
             </inertial>
         </link>
-        <link name="${prefix}link6_right_wrist">
+        <link name="${prefix}link6">
             <visual>
                 <!--J6 right_wrist/Part__Feature006.-->
-                <origin rpy="-2.1276679791326423 -1.5542266826921929 0" xyz="-0.0485412 -0.0860404 0.437784"/>
-                <geometry>
-                    <mesh filename="package://openarm_two_arms/meshes/full_upper_j6v1_mg9rps.dae"/>
+                <origin rpy="${reflect*-2.1276679791326423} ${rotate -1.5542266826921929} ${rotate}" xyz="-0.0485412 -0.0860404 0.437784"/>
+                <geometry>
+                    <mesh filename="package://openarm_two_arms/meshes/${'full_upper_j6v1_mg9rps.dae' if side=='right' else 'full_upper_j6_leftv005_f8km11.dae'}"/>
                 </geometry>
             </visual>
@@ -139,5 +139,5 @@
                 <origin rpy="0 -0.008758182894510852 0" xyz="0.558839 -0.00358671 -0.0631962"/>
                 <geometry>
-                    <mesh filename="package://openarm_two_arms/meshes/full_upper_j7v1_9yzky6.dae"/>
+                    <mesh filename="package://openarm_two_arms/meshes/${'full_upper_j7v1_9yzky6.dae' if side=='right' else 'full_upper_j7_leftv005_8ohvh2.dae'}"/>
                 </geometry>
             </visual>
@@ -248,5 +248,5 @@
         <joint name="${prefix}rev5" type="revolute">
             <parent link="${prefix}link5"/>
-            <child link="${prefix}link6_right_wrist"/>
+            <child link="${prefix}link6"/>
             <origin rpy="1.5707963267948473 -0.5569332500492129 1.556730325338251" xyz="-0.133937 0.00188408 -0.0297547"/>
             <axis xyz="0 0 1"/>
@@ -254,5 +254,5 @@
         </joint>
         <joint name="${prefix}rev6" type="revolute">
-            <parent link="${prefix}link6_right_wrist"/>
+            <parent link="${prefix}link6"/>
             <child link="${prefix}link7"/>
             <origin rpy="-1.5707963268024898 -1.5567303253382425 -0.5569332500461536" xyz="-0.0187648 -0.0301352 -0.12105"/>

Commit message: Add rotate mesh for actuator motor

File: openarm_two_arms/urdf/openarm.xacro (robot description, xacro)
@@ -116,5 +116,5 @@
             <visual>
                 <!--J6 right_wrist/Part__Feature006.-->
-                <origin rpy="${reflect*-2.1276679791326423} ${rotate -1.5542266826921929} ${rotate}" xyz="-0.0485412 -0.0860404 0.437784"/>
+                <origin rpy="${-2.1276679791326423 * reflect} ${reflect* -1.5542266826921929} 0" xyz="-0.0485412 -0.0860404 0.437784"/>
                 <geometry>
                     <mesh filename="package://openarm_two_arms/meshes/${'full_upper_j6v1_mg9rps.dae' if side=='right' else 'full_upper_j6_leftv005_f8km11.dae'}"/>
@@ -137,5 +137,5 @@
             <visual>
                 <!--J7 right v002/Part__Feature007.-->
-                <origin rpy="0 -0.008758182894510852 0" xyz="0.558839 -0.00358671 -0.0631962"/>
+                <origin rpy="0 ${reflect*-0.008758182894510852} 0" xyz="${reflect*0.558839} -0.00358671 -0.0631962"/>
                 <geometry>
                     <mesh filename="package://openarm_two_arms/meshes/${'full_upper_j7v1_9yzky6.dae' if side=='right' else 'full_upper_j7_leftv005_8ohvh2.dae'}"/>

Commit message: Close

File: openarm_two_arms/urdf/openarm.xacro (robot description, xacro)
@@ -116,5 +116,5 @@
             <visual>
                 <!--J6 right_wrist/Part__Feature006.-->
-                <origin rpy="${-2.1276679791326423 * reflect} ${reflect* -1.5542266826921929} 0" xyz="-0.0485412 -0.0860404 0.437784"/>
+                <origin rpy="-2.1276679791326423 ${reflect* -1.5542266826921929} 0" xyz="${reflect*-0.0485412} -0.0860404 0.437784"/>
                 <geometry>
                     <mesh filename="package://openarm_two_arms/meshes/${'full_upper_j6v1_mg9rps.dae' if side=='right' else 'full_upper_j6_leftv005_f8km11.dae'}"/>

Commit message: Complete mesh alignment for left arm

File: openarm_two_arms/urdf/openarm.xacro (robot description, xacro)
@@ -3,5 +3,4 @@
     <xacro:property name="side" value="right"/>
     <xacro:property name="prefix" value=""/>
-    <!-- <xacro:property name="pi" value="3.1415926535897927"/> -->
     <!-- <xacro:property name="zero_pos" value="vertical"/> -->
     <xacro:macro name="openarm" params="side prefix">
@@ -10,5 +9,4 @@
         <link name="${prefix}link1">
             <visual>
-                <!--J1 v002/Part__Feature001.-->
                 <origin rpy="0 0 0" xyz="0.0 0.0 -0.0007"/>
                 <geometry>
@@ -17,5 +15,4 @@
             </visual>
             <collision>
-                <!--bound_obj__right_link1__col_J1_v1__BoundBox/col_J1_v1__BoundBox.-->
                 <origin rpy="0 0 0" xyz="0.0 0.0 0.0289"/>
                 <geometry>
@@ -31,5 +28,4 @@
         <link name="${prefix}link2">
             <visual>
-                <!--J2 v002/Part__Feature002.-->
                 <origin rpy="0 0 0" xyz="0.0 0.0 -0.05395"/>
                 <geometry>
@@ -38,5 +34,4 @@
             </visual>
             <collision>
-                <!--bound_obj__right_link2__col_J2_v1__BoundBox/col_J2_v1__BoundBox.-->
                 <origin rpy="0 0 0" xyz="0.0 0.0 0.0371236"/>
                 <geometry>
@@ -52,5 +47,4 @@
         <link name="${prefix}link3">
             <visual>
-                <!--J3 v003/Part__Feature003.-->
                 <origin rpy="${pi * 0.5} 0 0" xyz="0.0 0.0987 0.02975"/>
                 <geometry>
@@ -59,5 +53,4 @@
             </visual>
             <collision>
-                <!--bound_obj__right_link3__col_J3_v2__BoundBox/col_J3_v2__BoundBox.-->
                 <origin rpy="${pi * 0.5} 0 0" xyz="-0.0164466 -0.00045542 0.02975"/>
                 <geometry>
@@ -73,5 +66,4 @@
         <link name="${prefix}link4">
             <visual>
-                <!--J4 v002/Part__Feature004.-->
                 <origin rpy="${pi} -1.5620381439005742 0" xyz="-0.0986962 0.0 0.0621144"/>
                 <geometry>
@@ -80,5 +72,4 @@
             </visual>
             <collision>
-                <!--bound_obj__right_link4__col_J4_v1__BoundBox/col_J4_v1__BoundBox.-->
                 <origin rpy="${pi} -1.5620381439005742 0" xyz="0.000266276 -0.0125642 -0.132604"/>
                 <geometry>
@@ -94,5 +85,4 @@
         <link name="${prefix}link5">
             <visual>
-                <!--J5 v003/Part__Feature005.-->
                 <origin rpy="0 -0.008758182894317394 0" xyz="0.303864 0.0 -0.128451"/>
                 <geometry>
@@ -101,5 +91,4 @@
             </visual>
             <collision>
-                <!--bound_obj__right_link5__col_J5_v2__BoundBox/col_J5_v2__BoundBox.-->
                 <origin rpy="0 -0.008758182894316818 0" xyz="-0.0542814 0.00265291 -0.0302022"/>
                 <geometry>
@@ -115,6 +104,5 @@
         <link name="${prefix}link6">
             <visual>
-                <!--J6 right_wrist/Part__Feature006.-->
-                <origin rpy="-2.1276679791326423 ${reflect* -1.5542266826921929} 0" xyz="${reflect*-0.0485412} -0.0860404 0.437784"/>
+                <origin rpy="${-2.1276679791326423*reflect + rotate} ${reflect* -1.5542266826921929} ${rotate}" xyz="${reflect*-0.0485412} ${reflect*-0.0860404} 0.437784"/>
                 <geometry>
                     <mesh filename="package://openarm_two_arms/meshes/${'full_upper_j6v1_mg9rps.dae' if side=='right' else 'full_upper_j6_leftv005_f8km11.dae'}"/>
@@ -122,5 +110,4 @@
             </visual>
             <collision>
-                <!--bound_obj__right_link6__col_J6_v1__BoundBox/col_J6_v1__BoundBox.-->
                 <origin rpy="-2.127667979132636 -1.5542266826921927 0" xyz="-0.00260794 -0.00312921 -0.0652641"/>
                 <geometry>
@@ -136,5 +123,4 @@
         <link name="${prefix}link7">
             <visual>
-                <!--J7 right v002/Part__Feature007.-->
                 <origin rpy="0 ${reflect*-0.008758182894510852} 0" xyz="${reflect*0.558839} -0.00358671 -0.0631962"/>
                 <geometry>
@@ -143,5 +129,4 @@
             </visual>
             <collision>
-                <!--bound_obj__right_link7__col_J7_v1__BoundBox/col_J7_v1__BoundBox.-->
                 <origin rpy="0 -0.008758182894511114 0" xyz="-0.000318103 0.0022839 0.0340014"/>
                 <geometry>
@@ -157,5 +142,4 @@
         <link name="${prefix}link8">
             <visual>
-                <!--J8 v002/Part__Feature008.-->
                 <origin rpy="1.5709195259578714 -0.014065461951077267 0" xyz="0.557948 0.103587 0.019724"/>
                 <geometry>
@@ -164,5 +148,4 @@
             </visual>
             <collision>
-                <!--bound_obj__right_link8__col_J8_v1__BoundBox/col_J8_v1__BoundBox.-->
                 <origin rpy="1.5709195259578714 -0.01406546195107726 0" xyz="-0.042694 -0.000543176 0.0110286"/>
                 <geometry>
@@ -178,5 +161,4 @@
         <link name="${prefix}link_left_jaw">
             <visual>
-                <!--left_jaw v002/Part__Feature009.-->
                 <origin rpy="0 -0.008758182894469432 0" xyz="0.665265 -0.00286677 -0.0209282"/>
                 <geometry>
@@ -185,5 +167,4 @@
             </visual>
             <collision>
-                <!--bound_obj__right_left_jaw__col_left_jaw_v1_col_obj/col_left_jaw_v1_col_obj.-->
                 <origin rpy="0 -0.0087581828944695 0" xyz="0.665265 -0.00286677 -0.0209282"/>
                 <geometry>
@@ -199,5 +180,4 @@
         <link name="${prefix}link_right_jaw">
             <visual>
-                <!--right_jaw v002/Part__Feature010.-->
                 <origin rpy="0 -0.008758182898001485 0" xyz="0.665265 -0.00286677 -0.175928"/>
                 <geometry>
@@ -206,5 +186,4 @@
             </visual>
             <collision>
-                <!--bound_obj__right_right_jaw__col_right_jaw_v1_col_obj/col_right_jaw_v1_col_obj.-->
                 <origin rpy="0 -0.008758182898001553 0" xyz="0.665265 -0.00286677 -0.175928"/>
                 <geometry>

File: openarm_two_arms/urdf/openarm_two_arms.urdf (robot description, URDF)
Before this commit: robot openarm_two_arms, 21 links, 20 joints
Links:
- removed link l_J1_v002
- removed link l_J2_v002
- removed link l_J2_v003
- removed link l_J3_v003
- removed link l_J3_v004
- removed link l_J4_v002
- removed link l_J4_v003
- removed link l_J5_v003
- removed link l_J5_v004
- removed link l_J6_Left_v004
- removed link l_J6_right_wrist
- removed link l_J7_Left_v004
- removed link l_J7_v002
- removed link l_J8_v002
- removed link l_J8_v003
- removed link l_base_link001
- removed link l_left_jaw_v002
- removed link l_left_jaw_v004
- removed link l_right_jaw_v002
- removed link l_right_jaw_v004
- added link left_link1, mass 0.5769283920617254; collision box size=0.11 0.073 0.0592; visual mesh filename=package://openarm_two_arms/meshes/full_upper_j1v1_fj2ul1.dae
- added link left_link2, mass 0.16257504134917358; collision box size=0.0590000000149012 0.08200000000000002 0.0742471498637348; visual mesh filename=package://openarm_two_arms/meshes/full_upper_j2v1_xzm1cu.dae
- added link left_link3, mass 0.4201676469910031; collision box size=0.08989101803441879 0.06999999999999983 0.05903276947803012; visual mesh filename=package://openarm_two_arms/meshes/full_upper_j3v2_5nirfo.dae
- added link left_link4, mass 0.819475539373447; collision box size=0.27584673777150337 0.08211429171582063 0.07186573179325861; visual mesh filename=package://openarm_two_arms/meshes/full_upper_j4v1_u1e2xn.dae
- added link left_link5, mass 0.4086748254352304; collision box size=0.16827213220625828 0.06430555048399171 0.08257859967140947; visual mesh filename=package://openarm_two_arms/meshes/full_upper_j5v2_ckk9an.dae
- added link left_link6, mass 0.3448471958049249; collision box size=0.13114353004704765 0.05953478325301745 0.08817196195081879; visual mesh filename=package://openarm_two_arms/meshes/full_upper_j6_leftv005_f8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
- added link left_link7, mass 0.2782138078738053; collision box size=0.058327402175132874 0.04432916698753661 0.08267601622411752; visual mesh filename=package://openarm_two_arms/meshes/full_upper_j7_leftv005_8o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
- added link left_link8, mass 0.31261452743802165; collision box size=0.13038799671743653 0.05180887692688926 0.1601236763440867; visual mesh filename=package://openarm_two_arms/meshes/full_upper_j8v1_dka5zq.dae
- added link left_link_left_jaw, mass 0.04297897856394934; collision mesh filename=package://openarm_two_arms/meshes/full_upper_col_left_jaw_v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; visual mesh filename=package://openarm_two_arms/meshes/full_upper_left_jawv1_6yx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
- added link left_link_right_jaw, mass 0.042981665301134515; collision mesh filename=package://openarm_two_arms/meshes/full_upper_col_right_jaw_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; visual mesh filename=package://openarm_two_arms/meshes/full_upper_right_jawv1_0f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
- added link right_link1, mass 0.5769283920617254; collision box size=0.11 0.073 0.0592; visual mesh filename=package://openarm_two_arms/meshes/full_upper_j1v1_fj2ul1.dae
- added link right_link2, mass 0.16257504134917358; collision box size=0.0590000000149012 0.08200000000000002 0.0742471498637348; visual mesh filename=package://openarm_two_arms/meshes/full_upper_j2v1_xzm1cu.dae
- added link right_link3, mass 0.4201676469910031; collision box size=0.08989101803441879 0.06999999999999983 0.05903276947803012; visual mesh filename=package://openarm_two_arms/meshes/full_upper_j3v2_5nirfo.dae
- added link right_link4, mass 0.819475539373447; collision box size=0.27584673777150337 0.08211429171582063 0.07186573179325861; visual mesh filename=package://openarm_two_arms/meshes/full_upper_j4v1_u1e2xn.dae
- added link right_link5, mass 0.4086748254352304; collision box size=0.16827213220625828 0.06430555048399171 0.08257859967140947; visual mesh filename=package://openarm_two_arms/meshes/full_upper_j5v2_ckk9an.dae
- added link right_link6, mass 0.3448471958049249; collision box size=0.13114353004704765 0.05953478325301745 0.08817196195081879; visual mesh filename=package://openarm_two_arms/meshes/full_upper_j6v1_mg9rps.dae
- added link right_link7, mass 0.2782138078738053; collision box size=0.058327402175132874 0.04432916698753661 0.08267601622411752; visual mesh filename=package://openarm_two_arms/meshes/full_upper_j7v1_9yzky6.dae
- added link right_link8, mass 0.31261452743802165; collision box size=0.13038799671743653 0.05180887692688926 0.1601236763440867; visual mesh filename=package://openarm_two_arms/meshes/full_upper_j8v1_dka5zq.dae
- added link right_link_left_jaw, mass 0.04297897856394934; collision mesh filename=package://openarm_two_arms/meshes/full_upper_col_left_jaw_v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; visual mesh filename=package://openarm_two_arms/meshes/full_upper_left_jawv1_6yx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
- added link right_link_right_jaw, mass 0.042981665301134515; collision mesh filename=package://openarm_two_arms/meshes/full_upper_col_right_jaw_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; visual mesh filename=package://openarm_two_arms/meshes/full_upper_right_jawv1_0f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
- added link world
Joints:
- added joint dummy_joint: type fixed, parent world, child pedestal_link, origin xyz=0.0 0.0 0.0 rpy=0.0 0.0 0.0
- joint left_fix1: child l_base_link001 -> right_link1; origin xyz=-0.09 0.0 0.893 rpy=3.0186531925068127 -1.5707963267948268 0.12293946108298068 -> xyz=-0.09 0.0 0.893 rpy=6.160245846096606 -1.5707963267948268 0.12293946108298068
- joint left_left_pris1: child l_left_jaw_v004 -> left_link_left_jaw; limit lower=-0.045 upper=0.0 effort=0.0 velocity=0.0 -> lower=0.0 upper=0.045 effort=0.0 velocity=0.0; origin xyz=0.10571 -0.0786733 0.0132053 rpy=1.5707963267947693 0.020777510312786344 -0.008760073612368274 -> xyz=-0.1071 0.0768568 0.0132053 rpy=1.570796326795101 -0.014066001454929162 0.00875904933542146; parent l_J8_v003 -> left_link8
- joint left_rev1: axis 0 0 1 -> 0 0 -1; child l_J2_v003 -> left_link2; origin xyz=0.0 0.0 -0.05325 rpy=-3.1415926535897922 0 -3.1415926535897927 -> xyz=0.0 0.0 0.05325 rpy=0 0 0; parent l_base_link001 -> left_link1
- joint left_rev2: child l_J3_v004 -> left_link3; limit lower=-3.141592653589793 upper=0.0 effort=0.0 velocity=0.0 -> lower=0.0 upper=3.141592653589793 effort=0.0 velocity=0.0; origin xyz=0.0 0.02975 0.04475 rpy=-1.570796326794897 0 0 -> xyz=0.0 -0.02975 0.04475 rpy=-1.5707963267948968 0 0; parent l_J2_v003 -> left_link2
- joint left_rev3: axis 0 0 1 -> 0 0 -1; child l_J4_v003 -> left_link4; origin xyz=0.0612477 -0.000536432 -0.02975 rpy=1.5707963267949063 0 1.5620381439005797 -> xyz=-0.0612477 -0.000536432 0.02975 rpy=-1.5707963267949054 3.141592653589793 -1.562038143900564; parent l_J3_v004 -> left_link3
- joint left_rev4: child l_J5_v004 -> left_link5; limit lower=-2.792526803190927 upper=0.3490658503988659 effort=0.0 velocity=0.0 -> lower=-0.3490658503988659 upper=2.792526803190927 effort=0.0 velocity=0.0; origin xyz=0.0297547 0.0 0.24175 rpy=-3.0383286058327292 -1.5707963267948855 3.038328605832587 -> xyz=0.0297547 0.0 -0.24175 rpy=-0.20701608758495998 -1.5707963267948566 -2.937419385117548; parent l_J4_v003 -> left_link4
- joint left_rev5: child l_J6_Left_v004 -> left_link6; origin xyz=0.133937 0.00188408 0.0297547 rpy=-1.5707963267949232 0.55693325005308 -1.5567303253382712 -> xyz=-0.133937 0.00188408 -0.0297547 rpy=1.5707963267948473 -0.5569332500492129 1.556730325338251; parent l_J5_v004 -> left_link5
- joint left_rev6: child l_J7_Left_v004 -> left_link7; origin xyz=0.0187648 0.0301352 0.12105 rpy=1.5707963267870033 -1.5567303253382319 -0.5569332500457352 -> xyz=-0.0187648 -0.0301352 -0.12105 rpy=-1.5707963268024898 -1.5567303253382425 -0.5569332500461536; parent l_J6_Left_v004 -> left_link6
- joint left_rev7: child l_J8_v003 -> left_link8; origin xyz=0.000320989 -0.0154467 0.0355 rpy=-1.5707963267949518 0.008760073613296379 0.020777510312798276 -> xyz=-0.000217313 -0.0154485 0.0355 rpy=-1.5707963267950005 -0.00875904933536772 -0.014066001454933467; parent l_J7_Left_v004 -> left_link7
- joint left_right_pris2: child l_right_jaw_v004 -> left_link_right_jaw; origin xyz=0.1071 0.0763207 0.0132053 rpy=1.5707963267948966 0.020777510312787576 -0.008760073613237863 -> xyz=-0.10571 -0.0781373 0.0132053 rpy=1.570796326794883 -0.014066001454927403 0.008759049336290027; parent l_J8_v003 -> left_link8
- joint right_fix1: child l_J1_v002 -> left_link1
- joint right_left_pris1: child l_left_jaw_v002 -> right_link_left_jaw; parent l_J8_v002 -> right_link8
- joint right_rev1: child l_J2_v002 -> right_link2; parent l_J1_v002 -> right_link1
- joint right_rev2: child l_J3_v003 -> right_link3; parent l_J2_v002 -> right_link2
- joint right_rev3: child l_J4_v002 -> right_link4; parent l_J3_v003 -> right_link3
- joint right_rev4: child l_J5_v003 -> right_link5; parent l_J4_v002 -> right_link4
- joint right_rev5: child l_J6_right_wrist -> right_link6; parent l_J5_v003 -> right_link5
- joint right_rev6: child l_J7_v002 -> right_link7; parent l_J6_right_wrist -> right_link6
- joint right_rev7: child l_J8_v002 -> right_link8; parent l_J7_v002 -> right_link7
- joint right_right_pris2: child l_right_jaw_v002 -> right_link_right_jaw; parent l_J8_v002 -> right_link8

File: openarm_two_arms/urdf/openarm_two_arms.urdf.xacro (robot description, xacro)
@@ -6,5 +6,4 @@
   <xacro:openarm prefix="right_" side="right"/>
   <xacro:openarm prefix="left_" side="left"/>
-  <!-- <xacro:include filename="openarm_left.urdf"/> -->
   <joint name="dummy_joint" type="fixed">
     <parent link="world"/>
@@ -12,12 +11,12 @@
     <origin xyz="0.0 0.0 0.0" rpy="0.0 0.0 0.0"/>
   </joint>
-  <joint name="right_fix1" type="fixed">
+  <joint name="right_fixed1" type="fixed">
+    <parent link="pedestal_link"/>
+    <child link="left_link1"/>
+    <origin rpy="3.0144791747751833 -1.5707963267948324 0.12689401604101067" xyz="0.09 0.0 0.893"/>
+  </joint>
+  <joint name="left_fixed1" type="fixed">
     <parent link="pedestal_link"/>
     <child link="right_link1"/>
-    <origin rpy="3.0144791747751833 -1.5707963267948324 0.12689401604101067" xyz="0.09 0.0 0.893"/>
-  </joint>
-  <joint name="left_fix1" type="fixed">
-    <parent link="pedestal_link"/>
-    <child link="left_link1"/>
     <origin rpy="${3.0186531925068127 + pi} -1.5707963267948268 0.12293946108298068" xyz="-0.09 0.0 0.893"/>
   </joint>

File: openarm_two_arms/urdf/openarm_two_arms_wrapper.urdf.xacro (robot description, xacro)
@@ -1,5 +1,5 @@
 <?xml version="1.0" encoding="utf-8"?>
 <robot xmlns:xacro="http://www.ros.org/wiki/xacro" name="openarm_two_arms">
-    <xacro:include filename="openarm_two_arms.urdf"/>
+    <xacro:include filename="openarm_two_arms.urdf.xacro"/>
     <xacro:include filename="openarm_two_arms_sensors.urdf.xacro"/>
 </robot>

Commit message: Align left arm mesh

File: openarm_two_arms/urdf/openarm.xacro (robot description, xacro)
@@ -104,5 +104,5 @@
         <link name="${prefix}link6">
             <visual>
-                <origin rpy="${-2.1276679791326423*reflect + rotate} ${reflect* -1.5542266826921929} ${rotate}" xyz="${reflect*-0.0485412} ${reflect*-0.0860404} 0.437784"/>
+                <origin rpy="${-2.1276679791326423*reflect + rotate} ${reflect* -1.5542266826921929} ${rotate}" xyz="${reflect*-0.0485412 + (0 if side=='right' else 0.012)} ${reflect*-0.0860404 +(0 if side=='right' else 0.0018)} ${0.437784- (0 if side=='right' else 0.0023)}"/>
                 <geometry>
                     <mesh filename="package://openarm_two_arms/meshes/${'full_upper_j6v1_mg9rps.dae' if side=='right' else 'full_upper_j6_leftv005_f8km11.dae'}"/>

Commit message: Align left gripper visual mesh

File: openarm_two_arms/urdf/openarm.xacro (robot description, xacro)
@@ -123,5 +123,5 @@
         <link name="${prefix}link7">
             <visual>
-                <origin rpy="0 ${reflect*-0.008758182894510852} 0" xyz="${reflect*0.558839} -0.00358671 -0.0631962"/>
+                <origin rpy="0 ${reflect*-0.008758182894510852 + rotate} 0" xyz="0.558839 ${reflect*-0.00358671 + (0 if side=='right' else -0.007)} ${reflect*-0.0631962 + (0 if side=='right' else 0.071)}"/>
                 <geometry>
                     <mesh filename="package://openarm_two_arms/meshes/${'full_upper_j7v1_9yzky6.dae' if side=='right' else 'full_upper_j7_leftv005_8ohvh2.dae'}"/>
