Commit message: Update rom of gripper to 4.51cm

File: openarm_two_arms/urdf/openarm.xacro (robot description, xacro)
@@ -251,5 +251,5 @@
             <origin rpy="1.570796326795101 -0.014066001454929162 0.00875904933542146" xyz="-0.1071 0.0768568 0.0132053"/>
             <axis xyz="0 0 1"/>
-            <limit effort="0.0" lower="0.0" upper="0.045" velocity="0.0"/>
+            <limit effort="0.0" lower="0.0" upper="0.0451" velocity="0.0"/>
         </joint>
         <joint name="${prefix}right_pris2" type="prismatic">
@@ -258,5 +258,5 @@
             <origin rpy="1.570796326794883 -0.014066001454927403 0.008759049336290027" xyz="-0.10571 -0.0781373 0.0132053"/>
             <axis xyz="0 0 1"/>
-            <limit effort="0.0" lower="0.0" upper="0.045" velocity="0.0"/>
+            <limit effort="0.0" lower="0.0" upper="0.0451" velocity="0.0"/>
             <mimic joint="${prefix}left_pris1" multiplier="-1.0" offset="0.0"/>
         </joint>

File: openarm_two_arms/urdf/openarm_two_arms.urdf (robot description, URDF)
Before this commit: robot openarm_two_arms, 22 links, 21 joints
Joints:
- joint left_left_pris1: limit lower=0.0 upper=0.045 effort=0.0 velocity=0.0 -> lower=0.0 upper=0.0451 effort=0.0 velocity=0.0
- joint left_right_pris2: limit lower=0.0 upper=0.045 effort=0.0 velocity=0.0 -> lower=0.0 upper=0.0451 effort=0.0 velocity=0.0
- joint right_left_pris1: limit lower=0.0 upper=0.045 effort=0.0 velocity=0.0 -> lower=0.0 upper=0.0451 effort=0.0 velocity=0.0
- joint right_right_pris2: limit lower=0.0 upper=0.045 effort=0.0 velocity=0.0 -> lower=0.0 upper=0.0451 effort=0.0 velocity=0.0

Commit message: Rename dae to more readable names

File: openarm_two_arms/urdf/openarm.xacro (robot description, xacro)
@@ -11,5 +11,5 @@
                 <origin rpy="0 0 0" xyz="0.0 0.0 -0.0007"/>
                 <geometry>
-                    <mesh filename="package://openarm_two_arms/meshes/full_upper_j1v1_fj2ul1.dae"/>
+                    <mesh filename="package://openarm_two_arms/meshes/link1.dae"/>
                 </geometry>
             </visual>
@@ -30,5 +30,5 @@
                 <origin rpy="0 0 0" xyz="0.0 0.0 -0.05395"/>
                 <geometry>
-                    <mesh filename="package://openarm_two_arms/meshes/full_upper_j2v1_xzm1cu.dae"/>
+                    <mesh filename="package://openarm_two_arms/meshes/link2.dae"/>
                 </geometry>
             </visual>
@@ -49,5 +49,5 @@
                 <origin rpy="${pi * 0.5} 0 0" xyz="0.0 0.0987 0.02975"/>
                 <geometry>
-                    <mesh filename="package://openarm_two_arms/meshes/full_upper_j3v2_5nirfo.dae"/>
+                    <mesh filename="package://openarm_two_arms/meshes/link3.dae"/>
                 </geometry>
             </visual>
@@ -68,5 +68,5 @@
                 <origin rpy="${pi} -1.5620381439005742 0" xyz="-0.0986962 0.0 0.0621144"/>
                 <geometry>
-                    <mesh filename="package://openarm_two_arms/meshes/full_upper_j4v1_u1e2xn.dae"/>
+                    <mesh filename="package://openarm_two_arms/meshes/link4.dae"/>
                 </geometry>
             </visual>
@@ -87,5 +87,5 @@
                 <origin rpy="0 -0.008758182894317394 0" xyz="0.303864 0.0 -0.128451"/>
                 <geometry>
-                    <mesh filename="package://openarm_two_arms/meshes/full_upper_j5v2_ckk9an.dae"/>
+                    <mesh filename="package://openarm_two_arms/meshes/link5.dae"/>
                 </geometry>
             </visual>
@@ -106,5 +106,5 @@
                 <origin rpy="${-2.1276679791326423*reflect + rotate} ${reflect* -1.5542266826921929} ${rotate}" xyz="${reflect*-0.0485412 + (0 if side=='right' else 0.012)} ${reflect*-0.0860404 +(0 if side=='right' else 0.0018)} ${0.437784- (0 if side=='right' else 0.0023)}"/>
                 <geometry>
-                    <mesh filename="package://openarm_two_arms/meshes/${'full_upper_j6v1_mg9rps.dae' if side=='right' else 'full_upper_j6_leftv005_f8km11.dae'}"/>
+                    <mesh filename="package://openarm_two_arms/meshes/${'link6_rightarm.dae' if side=='right' else 'link6_leftarm.dae'}"/>
                 </geometry>
             </visual>
@@ -125,5 +125,5 @@
                 <origin rpy="0 ${reflect*-0.008758182894510852 + rotate} 0" xyz="0.558839 ${reflect*-0.00358671 + (0 if side=='right' else -0.007)} ${reflect*-0.0631962 + (0 if side=='right' else 0.071)}"/>
                 <geometry>
-                    <mesh filename="package://openarm_two_arms/meshes/${'full_upper_j7v1_9yzky6.dae' if side=='right' else 'full_upper_j7_leftv005_8ohvh2.dae'}"/>
+                    <mesh filename="package://openarm_two_arms/meshes/${'link7_rightarm.dae' if side=='right' else 'link7_leftarm.dae'}"/>
                 </geometry>
             </visual>
@@ -144,5 +144,5 @@
                 <origin rpy="1.5709195259578714 -0.014065461951077267 0" xyz="0.557948 0.103587 0.019724"/>
                 <geometry>
-                    <mesh filename="package://openarm_two_arms/meshes/full_upper_j8v1_dka5zq.dae"/>
+                    <mesh filename="package://openarm_two_arms/meshes/link8.dae"/>
                 </geometry>
             </visual>
@@ -163,5 +163,5 @@
                 <origin rpy="0 -0.008758182894469432 0" xyz="0.665265 -0.00286677 -0.0209282"/>
                 <geometry>
-                    <mesh filename="package://openarm_two_arms/meshes/full_upper_left_jawv1_6yxtlc.dae"/>
+                    <mesh filename="package://openarm_two_arms/meshes/left_jaw.dae"/>
                 </geometry>
             </visual>
@@ -169,5 +169,5 @@
                 <origin rpy="0 -0.0087581828944695 0" xyz="0.665265 -0.00286677 -0.0209282"/>
                 <geometry>
-                    <mesh filename="package://openarm_two_arms/meshes/full_upper_col_left_jaw_v1_col_obj_wr4fju.dae"/>
+                    <mesh filename="package://openarm_two_arms/meshes/left_jaw.dae"/>
                 </geometry>
             </collision>
@@ -182,5 +182,5 @@
                 <origin rpy="0 -0.008758182898001485 0" xyz="0.665265 -0.00286677 -0.175928"/>
                 <geometry>
-                    <mesh filename="package://openarm_two_arms/meshes/full_upper_right_jawv1_0fmgsg.dae"/>
+                    <mesh filename="package://openarm_two_arms/meshes/right_jaw.dae"/>
                 </geometry>
             </visual>
@@ -188,5 +188,5 @@
                 <origin rpy="0 -0.008758182898001553 0" xyz="0.665265 -0.00286677 -0.175928"/>
                 <geometry>
-                    <mesh filename="package://openarm_two_arms/meshes/full_upper_col_right_jaw_v1_col_obj_9qatoq.dae"/>
+                    <mesh filename="package://openarm_two_arms/meshes/right_jaw.dae"/>
                 </geometry>
             </collision>

File: openarm_two_arms/urdf/openarm_two_arms.urdf (robot description, URDF)
Before this commit: robot openarm_two_arms, 22 links, 21 joints
Links:
- link left_link1: geometry collision box size=0.11 0.073 0.0592; visual mesh filename=package://openarm_two_arms/meshes/link1.dae
- link left_link2: geometry collision box size=0.0590000000149012 0.08200000000000002 0.0742471498637348; visual mesh filename=package://openarm_two_arms/meshes/link2.dae
- link left_link3: geometry collision box size=0.08989101803441879 0.06999999999999983 0.05903276947803012; visual mesh filename=package://openarm_two_arms/meshes/link3.dae
- link left_link4: geometry collision box size=0.27584673777150337 0.08211429171582063 0.07186573179325861; visual mesh filename=package://openarm_two_arms/meshes/link4.dae
- link left_link5: geometry collision box size=0.16827213220625828 0.06430555048399171 0.08257859967140947; visual mesh filename=package://openarm_two_arms/meshes/link5.dae
- link left_link6: geometry collision box size=0.13114353004704765 0.05953478325301745 0.08817196195081879; visual mesh filename=package://openarm_two_arms/meshes/link6_leftarm.dae
- link left_link7: geometry collision box size=0.058327402175132874 0.04432916698753661 0.08267601622411752; visual mesh filename=package://openarm_two_arms/meshes/link7_leftarm.dae
- link left_link8: geometry collision box size=0.13038799671743653 0.05180887692688926 0.1601236763440867; visual mesh filename=package://openarm_two_arms/meshes/link8.dae
- link left_link_left_jaw: geometry collision mesh filename=package://openarm_two_arms/meshes/left_jaw.dae; visual mesh filename=package://openarm_two_arms/meshes/left_jaw.dae
- link left_link_right_jaw: geometry collision mesh filename=package://openarm_two_arms/meshes/right_jaw.dae; visual mesh filename=package://openarm_two_arms/meshes/right_jaw.dae
- link pedestal_link: geometry collision box size=0.18 0.06 0.978000000000004; visual mesh filename=package://openarm_two_arms/meshes/pedestal_link.dae
- link right_link1: geometry collision box size=0.11 0.073 0.0592; visual mesh filename=package://openarm_two_arms/meshes/link1.dae
- link right_link2: geometry collision box size=0.0590000000149012 0.08200000000000002 0.0742471498637348; visual mesh filename=package://openarm_two_arms/meshes/link2.dae
- link right_link3: geometry collision box size=0.08989101803441879 0.06999999999999983 0.05903276947803012; visual mesh filename=package://openarm_two_arms/meshes/link3.dae
- link right_link4: geometry collision box size=0.27584673777150337 0.08211429171582063 0.07186573179325861; visual mesh filename=package://openarm_two_arms/meshes/link4.dae
- link right_link5: geometry collision box size=0.16827213220625828 0.06430555048399171 0.08257859967140947; visual mesh filename=package://openarm_two_arms/meshes/link5.dae
- link right_link6: geometry collision box size=0.13114353004704765 0.05953478325301745 0.08817196195081879; visual mesh filename=package://openarm_two_arms/meshes/link6_rightarm.dae
- link right_link7: geometry collision box size=0.058327402175132874 0.04432916698753661 0.08267601622411752; visual mesh filename=package://openarm_two_arms/meshes/link7_rightarm.dae
- link right_link8: geometry collision box size=0.13038799671743653 0.05180887692688926 0.1601236763440867; visual mesh filename=package://openarm_two_arms/meshes/link8.dae
- link right_link_left_jaw: geometry collision mesh filename=package://openarm_two_arms/meshes/left_jaw.dae; visual mesh filename=package://openarm_two_arms/meshes/left_jaw.dae
- link right_link_right_jaw: geometry collision mesh filename=package://openarm_two_arms/meshes/right_jaw.dae; visual mesh filename=package://openarm_two_arms/meshes/right_jaw.dae

File: openarm_two_arms/urdf/openarm_two_arms_pedestal.urdf (robot description, URDF)
Before this commit: robot openarm_two_arms, 1 links, 0 joints
Links:
- link pedestal_link: geometry collision box size=0.18 0.06 0.978000000000004; visual mesh filename=package://openarm_two_arms/meshes/pedestal_link.dae

Commit message: Use stl over dae

File: openarm_two_arms/urdf/openarm.xacro (robot description, xacro)
@@ -3,4 +3,7 @@
     <xacro:property name="side" value="right"/>
     <xacro:property name="prefix" value=""/>
+    <material name="gray">
+        <color rgba="${105/255} ${105/255} ${105/255} 1.0"/>
+    </material>
     <!-- <xacro:property name="zero_pos" value="vertical"/> -->
     <xacro:macro name="openarm" params="side prefix">
@@ -11,6 +14,7 @@
                 <origin rpy="0 0 0" xyz="0.0 0.0 -0.0007"/>
                 <geometry>
-                    <mesh filename="package://openarm_two_arms/meshes/link1.dae"/>
-                </geometry>
+                    <mesh filename="package://openarm_two_arms/meshes/link1.stl"/>
+                </geometry>
+                <material name="gray"/>
             </visual>
             <collision>
@@ -30,6 +34,7 @@
                 <origin rpy="0 0 0" xyz="0.0 0.0 -0.05395"/>
                 <geometry>
-                    <mesh filename="package://openarm_two_arms/meshes/link2.dae"/>
-                </geometry>
+                    <mesh filename="package://openarm_two_arms/meshes/link2.stl"/>
+                </geometry>
+                <material name="gray"/>
             </visual>
             <collision>
@@ -49,6 +54,7 @@
                 <origin rpy="${pi * 0.5} 0 0" xyz="0.0 0.0987 0.02975"/>
                 <geometry>
-                    <mesh filename="package://openarm_two_arms/meshes/link3.dae"/>
-                </geometry>
+                    <mesh filename="package://openarm_two_arms/meshes/link3.stl"/>
+                </geometry>
+                <material name="gray"/>
             </visual>
             <collision>
@@ -68,6 +74,7 @@
                 <origin rpy="${pi} -1.5620381439005742 0" xyz="-0.0986962 0.0 0.0621144"/>
                 <geometry>
-                    <mesh filename="package://openarm_two_arms/meshes/link4.dae"/>
-                </geometry>
+                    <mesh filename="package://openarm_two_arms/meshes/link4.stl"/>
+                </geometry>
+                <material name="gray"/>
             </visual>
             <collision>
@@ -87,6 +94,7 @@
                 <origin rpy="0 -0.008758182894317394 0" xyz="0.303864 0.0 -0.128451"/>
                 <geometry>
-                    <mesh filename="package://openarm_two_arms/meshes/link5.dae"/>
-                </geometry>
+                    <mesh filename="package://openarm_two_arms/meshes/link5.stl"/>
+                </geometry>
+                <material name="gray"/>
             </visual>
             <collision>
@@ -106,6 +114,7 @@
                 <origin rpy="${-2.1276679791326423*reflect + rotate} ${reflect* -1.5542266826921929} ${rotate}" xyz="${reflect*-0.0485412 + (0 if side=='right' else 0.012)} ${reflect*-0.0860404 +(0 if side=='right' else 0.0018)} ${0.437784- (0 if side=='right' else 0.0023)}"/>
                 <geometry>
-                    <mesh filename="package://openarm_two_arms/meshes/${'link6_rightarm.dae' if side=='right' else 'link6_leftarm.dae'}"/>
-                </geometry>
+                    <mesh filename="package://openarm_two_arms/meshes/${'link6_rightarm.stl' if side=='right' else 'link6_leftarm.stl'}"/>
+                </geometry>
+                <material name="gray"/>
             </visual>
             <collision>
@@ -125,6 +134,7 @@
                 <origin rpy="0 ${reflect*-0.008758182894510852 + rotate} 0" xyz="0.558839 ${reflect*-0.00358671 + (0 if side=='right' else -0.007)} ${reflect*-0.0631962 + (0 if side=='right' else 0.071)}"/>
                 <geometry>
-                    <mesh filename="package://openarm_two_arms/meshes/${'link7_rightarm.dae' if side=='right' else 'link7_leftarm.dae'}"/>
-                </geometry>
+                    <mesh filename="package://openarm_two_arms/meshes/${'link7_rightarm.stl' if side=='right' else 'link7_leftarm.stl'}"/>
+                </geometry>
+                <material name="gray"/>
             </visual>
             <collision>
@@ -144,6 +154,7 @@
                 <origin rpy="1.5709195259578714 -0.014065461951077267 0" xyz="0.557948 0.103587 0.019724"/>
                 <geometry>
-                    <mesh filename="package://openarm_two_arms/meshes/link8.dae"/>
-                </geometry>
+                    <mesh filename="package://openarm_two_arms/meshes/link8.stl"/>
+                </geometry>
+                <material name="gray"/>
             </visual>
             <collision>
@@ -163,11 +174,12 @@
                 <origin rpy="0 -0.008758182894469432 0" xyz="0.665265 -0.00286677 -0.0209282"/>
                 <geometry>
-                    <mesh filename="package://openarm_two_arms/meshes/left_jaw.dae"/>
-                </geometry>
+                    <mesh filename="package://openarm_two_arms/meshes/left_jaw.stl"/>
+                </geometry>
+                <material name="gray"/>
             </visual>
             <collision>
                 <origin rpy="0 -0.0087581828944695 0" xyz="0.665265 -0.00286677 -0.0209282"/>
                 <geometry>
-                    <mesh filename="package://openarm_two_arms/meshes/left_jaw.dae"/>
+                    <mesh filename="package://openarm_two_arms/meshes/left_jaw.stl"/>
                 </geometry>
             </collision>
@@ -182,11 +194,12 @@
                 <origin rpy="0 -0.008758182898001485 0" xyz="0.665265 -0.00286677 -0.175928"/>
                 <geometry>
-                    <mesh filename="package://openarm_two_arms/meshes/right_jaw.dae"/>
-                </geometry>
+                    <mesh filename="package://openarm_two_arms/meshes/right_jaw.stl"/>
+                </geometry>
+                <material name="gray"/>
             </visual>
             <collision>
                 <origin rpy="0 -0.008758182898001553 0" xyz="0.665265 -0.00286677 -0.175928"/>
                 <geometry>
-                    <mesh filename="package://openarm_two_arms/meshes/right_jaw.dae"/>
+                    <mesh filename="package://openarm_two_arms/meshes/right_jaw.stl"/>
                 </geometry>
             </collision>

File: openarm_two_arms/urdf/openarm_two_arms.urdf (robot description, URDF)
Before this commit: robot openarm_two_arms, 22 links, 21 joints
Links:
- link left_link1: geometry collision box size=0.11 0.073 0.0592; visual mesh filename=package://openarm_two_arms/meshes/link1.stl
- link left_link2: geometry collision box size=0.0590000000149012 0.08200000000000002 0.0742471498637348; visual mesh filename=package://openarm_two_arms/meshes/link2.stl
- link left_link3: geometry collision box size=0.08989101803441879 0.06999999999999983 0.05903276947803012; visual mesh filename=package://openarm_two_arms/meshes/link3.stl
- link left_link4: geometry collision box size=0.27584673777150337 0.08211429171582063 0.07186573179325861; visual mesh filename=package://openarm_two_arms/meshes/link4.stl
- link left_link5: geometry collision box size=0.16827213220625828 0.06430555048399171 0.08257859967140947; visual mesh filename=package://openarm_two_arms/meshes/link5.stl
- link left_link6: geometry collision box size=0.13114353004704765 0.05953478325301745 0.08817196195081879; visual mesh filename=package://openarm_two_arms/meshes/link6_leftarm.stl
- link left_link7: geometry collision box size=0.058327402175132874 0.04432916698753661 0.08267601622411752; visual mesh filename=package://openarm_two_arms/meshes/link7_leftarm.stl
- link left_link8: geometry collision box size=0.13038799671743653 0.05180887692688926 0.1601236763440867; visual mesh filename=package://openarm_two_arms/meshes/link8.stl
- link left_link_left_jaw: geometry collision mesh filename=package://openarm_two_arms/meshes/left_jaw.stl; visual mesh filename=package://openarm_two_arms/meshes/left_jaw.stl
- link left_link_right_jaw: geometry collision mesh filename=package://openarm_two_arms/meshes/right_jaw.stl; visual mesh filename=package://openarm_two_arms/meshes/right_jaw.stl
- link pedestal_link: geometry collision box size=0.18 0.06 0.978000000000004; visual mesh filename=package://openarm_two_arms/meshes/pedestal_link.stl
- link right_link1: geometry collision box size=0.11 0.073 0.0592; visual mesh filename=package://openarm_two_arms/meshes/link1.stl
- link right_link2: geometry collision box size=0.0590000000149012 0.08200000000000002 0.0742471498637348; visual mesh filename=package://openarm_two_arms/meshes/link2.stl
- link right_link3: geometry collision box size=0.08989101803441879 0.06999999999999983 0.05903276947803012; visual mesh filename=package://openarm_two_arms/meshes/link3.stl
- link right_link4: geometry collision box size=0.27584673777150337 0.08211429171582063 0.07186573179325861; visual mesh filename=package://openarm_two_arms/meshes/link4.stl
- link right_link5: geometry collision box size=0.16827213220625828 0.06430555048399171 0.08257859967140947; visual mesh filename=package://openarm_two_arms/meshes/link5.stl
- link right_link6: geometry collision box size=0.13114353004704765 0.05953478325301745 0.08817196195081879; visual mesh filename=package://openarm_two_arms/meshes/link6_rightarm.stl
- link right_link7: geometry collision box size=0.058327402175132874 0.04432916698753661 0.08267601622411752; visual mesh filename=package://openarm_two_arms/meshes/link7_rightarm.stl
- link right_link8: geometry collision box size=0.13038799671743653 0.05180887692688926 0.1601236763440867; visual mesh filename=package://openarm_two_arms/meshes/link8.stl
- link right_link_left_jaw: geometry collision mesh filename=package://openarm_two_arms/meshes/left_jaw.stl; visual mesh filename=package://openarm_two_arms/meshes/left_jaw.stl
- link right_link_right_jaw: geometry collision mesh filename=package://openarm_two_arms/meshes/right_jaw.stl; visual mesh filename=package://openarm_two_arms/meshes/right_jaw.stl

File: openarm_two_arms/urdf/openarm_two_arms_pedestal.urdf (robot description, URDF)
Before this commit: robot openarm_two_arms, 1 links, 0 joints
Links:
- link pedestal_link: geometry collision box size=0.18 0.06 0.978000000000004; visual mesh filename=package://openarm_two_arms/meshes/pedestal_link.stl
