Commit message: Add openarm_bimanual_moveit_config and deploy to physical openarm (#3)
See https://github.com/reazon-research/openarm_ros2/pull/3 for video

File: openarm_bimanual_description/urdf/openarm_bimanual.urdf (robot description, URDF)
Before this commit: robot openarm_bimanual, 22 links, 21 joints
Links:
- added link camera_accel_frame
- added link camera_accel_optical_frame
- added link camera_bottom_screw_frame
- added link camera_color_frame
- added link camera_color_optical_frame
- added link camera_depth_frame
- added link camera_depth_optical_frame
- added link camera_gyro_frame
- added link camera_gyro_optical_frame
- added link camera_infra1_frame
- added link camera_infra1_optical_frame
- added link camera_infra2_frame
- added link camera_infra2_optical_frame
- added link camera_link, mass 0.072; collision box size=0.02505 0.09 0.025; visual mesh filename=file:///opt/ros/humble/share/realsense2_description/meshes/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
- added link left_dummy_link
- added link right_dummy_link
Joints:
- added joint camera_accel_joint: type fixed, parent camera_link, child camera_accel_frame, origin xyz=-0.01174 -0.00552 0.0051 rpy=0 0 0
- added joint camera_accel_optical_joint: type fixed, parent camera_accel_frame, child camera_accel_optical_frame, origin xyz=0 0 0 rpy=-1.5707963267948966 0 -1.5707963267948966
- added joint camera_color_joint: type fixed, parent camera_link, child camera_color_frame, origin xyz=0 0.015 0 rpy=0 0 0
- added joint camera_color_optical_joint: type fixed, parent camera_color_frame, child camera_color_optical_frame, origin xyz=0 0 0 rpy=-1.5707963267948966 0 -1.5707963267948966
- added joint camera_depth_joint: type fixed, parent camera_link, child camera_depth_frame, origin xyz=0 0 0 rpy=0 0 0
- added joint camera_depth_optical_joint: type fixed, parent camera_depth_frame, child camera_depth_optical_frame, origin xyz=0 0 0 rpy=-1.5707963267948966 0 -1.5707963267948966
- added joint camera_gyro_joint: type fixed, parent camera_link, child camera_gyro_frame, origin xyz=-0.01174 -0.00552 0.0051 rpy=0 0 0
- added joint camera_gyro_optical_joint: type fixed, parent camera_gyro_frame, child camera_gyro_optical_frame, origin xyz=0 0 0 rpy=-1.5707963267948966 0 -1.5707963267948966
- added joint camera_infra1_joint: type fixed, parent camera_link, child camera_infra1_frame, origin xyz=0 0.0 0 rpy=0 0 0
- added joint camera_infra1_optical_joint: type fixed, parent camera_infra1_frame, child camera_infra1_optical_frame, origin xyz=0 0 0 rpy=-1.5707963267948966 0 -1.5707963267948966
- added joint camera_infra2_joint: type fixed, parent camera_link, child camera_infra2_frame, origin xyz=0 -0.05 0 rpy=0 0 0
- added joint camera_infra2_optical_joint: type fixed, parent camera_infra2_frame, child camera_infra2_optical_frame, origin xyz=0 0 0 rpy=-1.5707963267948966 0 -1.5707963267948966
- added joint camera_joint: type fixed, parent pedestal_link, child camera_bottom_screw_frame, origin xyz=0.0 -0.025 0.995216 rpy=0.0 0.0 -1.5707963267948966
- added joint camera_link_joint: type fixed, parent camera_bottom_screw_frame, child camera_link, origin xyz=0.010600000000000002 0.0175 0.0125 rpy=0 0 0
- added joint left_dummy_joint: type fixed, parent left_dummy_link, child left_link1
- added joint right_dummy_joint: type fixed, parent right_dummy_link, child right_link1
- joint left_fixed1: child right_link1 -> left_dummy_link; origin xyz=-0.09 0.0 0.893 rpy=6.160245846096606 -1.5707963267948268 0.12293946108298068 -> xyz=0.09 0.0 0.893 rpy=3.0144791747751833 -1.5707963267948324 0.12689401604101067
- joint left_left_pris1: limit lower=0.0 upper=0.0451 effort=0.0 velocity=0.0 -> lower=-0.0451 upper=0.0 effort=0.0 velocity=0.0
- joint left_rev5: axis 0 0 1 -> 0 0 -1
- joint left_rev7: axis 0 0 1 -> 0 0 -1
- joint left_right_pris2: limit lower=0.0 upper=0.0451 effort=0.0 velocity=0.0 -> lower=-0.0451 upper=0.0 effort=0.0 velocity=0.0
- joint right_fixed1: child left_link1 -> right_dummy_link; origin xyz=0.09 0.0 0.893 rpy=3.0144791747751833 -1.5707963267948324 0.12689401604101067 -> xyz=-0.09 0.0 0.893 rpy=6.160245846096606 -1.5707963267948268 0.12293946108298068
- joint right_left_pris1: limit lower=0.0 upper=0.0451 effort=0.0 velocity=0.0 -> lower=-0.0451 upper=0.0 effort=0.0 velocity=0.0
- joint right_rev3: axis 0 0 1 -> 0 0 -1
- joint right_rev5: axis 0 0 1 -> 0 0 -1
- joint right_rev7: axis 0 0 1 -> 0 0 -1
- joint right_right_pris2: limit lower=0.0 upper=0.0451 effort=0.0 velocity=0.0 -> lower=-0.0451 upper=0.0 effort=0.0 velocity=0.0

File: openarm_bimanual_description/urdf/openarm_bimanual.urdf.xacro (robot description, xacro)
@@ -1,9 +1,8 @@
 <?xml version="1.0" ?>
 <robot xmlns:xacro="http://www.ros.org/wiki/xacro" name="openarm_bimanual">
-  <link name="world"/>
   <xacro:include filename="$(find openarm_description)/urdf/openarm.xacro"/>
   <xacro:include filename="openarm_pedestal.urdf"/>
-  <xacro:openarm prefix="right_" side="right" zero_pos="arm"/>
-  <xacro:openarm prefix="left_" side="left" zero_pos="arm"/>
+  <xacro:include filename="openarm_bimanual_sensors.xacro"/>
+  <link name="world"/>
   <joint name="dummy_joint" type="fixed">
     <parent link="world"/>
@@ -11,13 +10,15 @@
     <origin xyz="0.0 0.0 0.0" rpy="0.0 0.0 0.0"/>
   </joint>
+  <xacro:openarm prefix="right_" side="right" zero_pos="arm" can_device="can0"/>
+  <joint name="right_fixed1" type="fixed">
+    <parent link="pedestal_link"/>
+    <child link="right_dummy_link"/>
+    <origin rpy="${3.0186531925068127 + pi} -1.5707963267948268 0.12293946108298068" xyz="-0.09 0.0 0.893"/>
+  </joint>
+  <xacro:openarm prefix="left_" side="left" zero_pos="arm" can_device="can1"/>
   <joint name="left_fixed1" type="fixed">
     <parent link="pedestal_link"/>
-    <child link="left_link1"/>
+    <child link="left_dummy_link"/>
     <origin rpy="3.0144791747751833 -1.5707963267948324 0.12689401604101067" xyz="0.09 0.0 0.893"/>
   </joint>
-  <joint name="right_fixed1" type="fixed">
-    <parent link="pedestal_link"/>
-    <child link="right_link1"/>
-    <origin rpy="${3.0186531925068127 + pi} -1.5707963267948268 0.12293946108298068" xyz="-0.09 0.0 0.893"/>
-  </joint>
 </robot>

File: openarm_bimanual_description/urdf/openarm_bimanual_sensors.xacro (robot description, xacro)
@@ -1,3 +1,7 @@
 <?xml version="1.0"?>
 <robot xmlns:xacro="http://www.ros.org/wiki/xacro">
+    <xacro:include filename="$(find realsense2_description)/urdf/_d435i.urdf.xacro"/>
+    <xacro:sensor_d435i parent="pedestal_link" use_nominal_extrinsics="true">
+        <origin xyz="0.0 -0.025 0.995216" rpy="0.0 0.0 ${-pi/2.0}"/>
+    </xacro:sensor_d435i>
 </robot>

File: openarm_description/urdf/openarm.ros2_control.xacro (robot description, xacro)
@@ -1,11 +1,13 @@
 <?xml version="1.0"?>
 <robot xmlns:xacro="http://www.ros.org/wiki/xacro">
-    <xacro:macro name="openarm_ros2_control" params="name initial_positions_file prefix:=''">
+    <xacro:macro name="openarm_ros2_control" params="name initial_positions_file prefix:='' can_device='can0'">
         <xacro:property name="initial_positions" value="${xacro.load_yaml(initial_positions_file)['initial_positions']}"/>
         <ros2_control name="${prefix}${name}" type="system">
             <hardware>
                 <!-- By default, set up controllers for simulation. This won't work on real hardware -->
-                <plugin>mock_components/GenericSystem</plugin>
+                <!-- <plugin>mock_components/GenericSystem</plugin> -->
                 <plugin>openarm_hardware/OpenArmHW</plugin>
+                <param name="prefix">${prefix}</param>
+                <param name="can_device">${can_device}</param>
             </hardware>
             <joint name="${prefix}rev1">
@@ -13,7 +15,5 @@
                 <command_interface name="velocity"/>
                 <command_interface name="effort"/>
-                <state_interface name="position">
-                  <param name="initial_value">${initial_positions['rev1']}</param>
-                </state_interface>
+                <state_interface name="position"/>
                 <state_interface name="velocity"/>
                 <state_interface name="effort"/>
@@ -23,7 +23,5 @@
                 <command_interface name="velocity"/>
                 <command_interface name="effort"/>
-                <state_interface name="position">
-                  <param name="initial_value">${initial_positions['rev2']}</param>
-                </state_interface>
+                <state_interface name="position"/>
                 <state_interface name="velocity"/>
                 <state_interface name="effort"/>
@@ -33,7 +31,5 @@
                 <command_interface name="velocity"/>
                 <command_interface name="effort"/>
-                <state_interface name="position">
-                  <param name="initial_value">${initial_positions['rev3']}</param>
-                </state_interface>
+                <state_interface name="position"/>
                 <state_interface name="velocity"/>
                 <state_interface name="effort"/>
@@ -43,7 +39,5 @@
                 <command_interface name="velocity"/>
                 <command_interface name="effort"/>
-                <state_interface name="position">
-                  <param name="initial_value">${initial_positions['rev4']}</param>
-                </state_interface>
+                <state_interface name="position"/>
                 <state_interface name="velocity"/>
                 <state_interface name="effort"/>
@@ -53,7 +47,5 @@
                 <command_interface name="velocity"/>
                 <command_interface name="effort"/>
-                <state_interface name="position">
-                  <param name="initial_value">${initial_positions['rev5']}</param>
-                </state_interface>
+                <state_interface name="position"/>
                 <state_interface name="velocity"/>
                 <state_interface name="effort"/>
@@ -63,7 +55,5 @@
                 <command_interface name="velocity"/>
                 <command_interface name="effort"/>
-                <state_interface name="position">
-                  <param name="initial_value">${initial_positions['rev6']}</param>
-                </state_interface>
+                <state_interface name="position"/>
                 <state_interface name="velocity"/>
                 <state_interface name="effort"/>
@@ -73,7 +63,5 @@
                 <command_interface name="velocity"/>
                 <command_interface name="effort"/>
-                <state_interface name="position">
-                  <param name="initial_value">${initial_positions['rev7']}</param>
-                </state_interface>
+                <state_interface name="position"/>
                 <state_interface name="velocity"/>
                 <state_interface name="effort"/>
@@ -81,14 +69,12 @@
             <joint name="${prefix}left_pris1">
                 <command_interface name="position"/>
-                <state_interface name="position">
-                  <param name="initial_value">${initial_positions['left_pris1']}</param>
-                </state_interface>
+                <state_interface name="position"/>
                 <state_interface name="velocity"/>
             </joint>
-            <joint name="${prefix}right_pris2">
+            <!-- <joint name="${prefix}right_pris2">
                 <state_interface name="position">
-                  <param name="initial_value">${initial_positions['left_pris1']}</param>
+                  <param name="initial_value">${initial_positions['right_pris2']}</param>
                 </state_interface>
-            </joint>
+            </joint> -->
         </ros2_control>
     </xacro:macro>

File: openarm_description/urdf/openarm.urdf.xacro (robot description, xacro)
@@ -3,6 +3,4 @@
     <xacro:include filename="openarm.xacro"/>
     <xacro:openarm/>
-    <xacro:include filename="openarm_sensors.xacro"/>
-    <xacro:include filename="openarm.ros2_control.xacro" />
-    <xacro:openarm_ros2_control name="OpenArmHW" prefix="${prefix}" initial_positions_file="$(arg initial_positions_file)"/>
+    <xacro:include filename="$(find openarm_description)/urdf/openarm_sensors.xacro"/>
 </robot>

File: openarm_description/urdf/openarm.xacro (robot description, xacro)
@@ -4,5 +4,8 @@
         <color rgba="${105/255} ${105/255} ${105/255} 1.0"/>
     </material>
-    <xacro:macro name="openarm" params="side:='right' prefix:='' zero_pos='up'">
+    <material name="dark_gray">
+        <color rgba="${50/255} ${50/255} ${50/255} 1.0"/>
+    </material>
+    <xacro:macro name="openarm" params="side:='right' prefix:='' zero_pos='up' can_device='can0'">
         <!-- side right, left -->
         <!-- recommended prefixes left_, right_, etc. -->
@@ -10,5 +13,12 @@
         <xacro:property name="reflect" value="${1 if side=='right' else -1}"/>
         <xacro:property name="rotate" value="${0 if side=='right' else pi}"/>
-        <xacro:arg name="initial_positions_file" default="initial_positions.yaml" />
+        <xacro:include filename="$(find openarm_description)/urdf/openarm.ros2_control.xacro" />
+        <xacro:arg name="initial_positions_file" default="$(find openarm_description)/config/initial_positions.yaml" />
+        <xacro:openarm_ros2_control name="OpenArmHW" prefix="${prefix}" initial_positions_file="$(arg initial_positions_file)" can_device="${can_device}"/>
+        <link name="${prefix}dummy_link"/>
+        <joint name="${prefix}dummy_joint" type="fixed">
+            <parent link="${prefix}dummy_link"/>
+            <child link="${prefix}link1"/>
+        </joint>
         <link name="${prefix}link1">
             <visual>
@@ -215,5 +225,5 @@
             <child link="${prefix}link2"/>
             <origin rpy="0 0 0" xyz="0.0 0.0 0.05325"/>
-            <axis xyz="0 0 ${reflect*1}"/>
+            <axis xyz="0 0 1"/>
             <limit effort="0.0" lower="-2.0943951023931953" upper="2.0943951023931953" velocity="0.0"/>
         </joint>
@@ -221,7 +231,7 @@
             <parent link="${prefix}link2"/>
             <child link="${prefix}link3"/>
-            <origin rpy="-1.5707963267948968 ${pi/2 if zero_pos=='up' else 0} 0" xyz="0.0 -0.02975 0.04475"/>
-            <axis xyz="0 0 1"/>
-            <limit effort="0.0" lower="${-pi/2.0 if zero_pos=='up' else 0.0}" upper="${pi/2 if zero_pos=='up' else pi}" velocity="0.0"/>
+            <origin rpy="-1.5707963267948968 ${pi/2 if zero_pos=='up' else 0.0} 0.0" xyz="0.0 -0.02975 0.04475"/>
+            <axis xyz="0 0 ${reflect * -1}"/>
+            <limit effort="0.0" lower="${-pi/2.0 if zero_pos=='up' else -pi + rotate}" upper="${pi/2 if zero_pos=='up' else 0 + rotate}" velocity="0.0"/>
         </joint>
         <joint name="${prefix}rev3" type="revolute">
@@ -229,5 +239,5 @@
             <child link="${prefix}link4"/>
             <origin rpy="-1.5707963267949054 ${rotate} -1.562038143900564" xyz="-0.0612477 -0.000536432 0.02975"/>
-            <axis xyz="0 0 ${reflect*1}"/>
+            <axis xyz="0 0 -1"/>
             <limit effort="0.0" lower="-3.6651914291880923" upper="0.5235987755982988" velocity="0.0"/>
         </joint>
@@ -243,5 +253,5 @@
             <child link="${prefix}link6"/>
             <origin rpy="1.5707963267948473 -0.5569332500492129 1.556730325338251" xyz="-0.133937 0.00188408 -0.0297547"/>
-            <axis xyz="0 0 1"/>
+            <axis xyz="0 0 -1"/>
             <limit effort="0.0" lower="-2.0943951023931953" upper="2.0943951023931953" velocity="0.0"/>
         </joint>
@@ -250,5 +260,5 @@
             <child link="${prefix}link7"/>
             <origin rpy="-1.5707963268024898 -1.5567303253382425 -0.5569332500461536" xyz="-0.0187648 -0.0301352 -0.12105"/>
-            <axis xyz="0 0 1"/>
+            <axis xyz="0 0 ${reflect}"/>
             <limit effort="0.0" lower="-1.5707963267948966" upper="1.5707963267948966" velocity="0.0"/>
         </joint>
@@ -257,5 +267,5 @@
             <child link="${prefix}link8"/>
             <origin rpy="-1.5707963267950005 -0.00875904933536772 -0.014066001454933467" xyz="-0.000217313 -0.0154485 0.0355"/>
-            <axis xyz="0 0 1"/>
+            <axis xyz="0 0 -1"/>
             <limit effort="0.0" lower="-0.9599310885968813" upper="0.9599310885968813" velocity="0.0"/>
         </joint>
@@ -265,5 +275,5 @@
             <origin rpy="1.570796326795101 -0.014066001454929162 0.00875904933542146" xyz="-0.1071 0.0768568 0.0132053"/>
             <axis xyz="0 0 1"/>
-            <limit effort="0.0" lower="0.0" upper="0.0451" velocity="0.0"/>
+            <limit effort="0.0" lower="-0.0451" upper="0.0" velocity="0.0"/>
         </joint>
         <joint name="${prefix}right_pris2" type="prismatic">
@@ -272,5 +282,5 @@
             <origin rpy="1.570796326794883 -0.014066001454927403 0.008759049336290027" xyz="-0.10571 -0.0781373 0.0132053"/>
             <axis xyz="0 0 1"/>
-            <limit effort="0.0" lower="0.0" upper="0.0451" velocity="0.0"/>
+            <limit effort="0.0" lower="-0.0451" upper="0.0" velocity="0.0"/>
             <mimic joint="${prefix}left_pris1" multiplier="-1.0" offset="0.0"/>
         </joint>

Commit message: Add URDFs

File: openarm_bimanual_description/urdf/openarm_bimanual.urdf (robot description, URDF)
Before this commit: robot openarm_bimanual, 38 links, 37 joints
Links:
- removed link camera_accel_frame
- removed link camera_accel_optical_frame
- removed link camera_bottom_screw_frame
- removed link camera_color_frame
- removed link camera_color_optical_frame
- removed link camera_depth_frame
- removed link camera_depth_optical_frame
- removed link camera_gyro_frame
- removed link camera_gyro_optical_frame
- removed link camera_infra1_frame
- removed link camera_infra1_optical_frame
- removed link camera_infra2_frame
- removed link camera_infra2_optical_frame
- removed link camera_link
- added link left_gripper_center
- added link right_gripper_center
Joints:
- removed joint camera_accel_joint
- removed joint camera_accel_optical_joint
- removed joint camera_color_joint
- removed joint camera_color_optical_joint
- removed joint camera_depth_joint
- removed joint camera_depth_optical_joint
- removed joint camera_gyro_joint
- removed joint camera_gyro_optical_joint
- removed joint camera_infra1_joint
- removed joint camera_infra1_optical_joint
- removed joint camera_infra2_joint
- removed joint camera_infra2_optical_joint
- removed joint camera_joint
- removed joint camera_link_joint
- added joint left_virtual_gripper_center: type fixed, parent left_link8, child left_gripper_center, origin xyz=-0.13 0.00 0.0132053 rpy=0 0 0
- added joint right_virtual_gripper_center: type fixed, parent right_link8, child right_gripper_center, origin xyz=-0.13 0.00 0.0132053 rpy=0 0 0
- joint left_rev1: axis 0 0 -1 -> 0 0 1
- joint left_rev2: origin xyz=0.0 -0.02975 0.04475 rpy=-1.5707963267948968 0 0 -> xyz=0.0 -0.02975 0.04475 rpy=-1.5707963267948968 0.0 0.0
- joint left_rev6: axis 0 0 1 -> 0 0 -1
- joint right_rev2: axis 0 0 1 -> 0 0 -1; limit lower=0.0 upper=3.141592653589793 effort=0.0 velocity=0.0 -> lower=-3.141592653589793 upper=0 effort=0.0 velocity=0.0; origin xyz=0.0 -0.02975 0.04475 rpy=-1.5707963267948968 0 0 -> xyz=0.0 -0.02975 0.04475 rpy=-1.5707963267948968 0.0 0.0

File: openarm_bimanual_description/urdf/openarm_bimanual.urdf.xacro (robot description, xacro)
@@ -3,5 +3,5 @@
   <xacro:include filename="$(find openarm_description)/urdf/openarm.xacro"/>
   <xacro:include filename="openarm_pedestal.urdf"/>
-  <xacro:include filename="openarm_bimanual_sensors.xacro"/>
+  <!-- <xacro:include filename="openarm_bimanual_sensors.xacro"/> -->
   <link name="world"/>
   <joint name="dummy_joint" type="fixed">

File: openarm_description/urdf/openarm.urdf (robot description, URDF)
Before this commit: robot openarm, 11 links, 10 joints
Links:
- added link gripper_center
Joints:
- added joint virtual_gripper_center: type fixed, parent link8, child gripper_center, origin xyz=-0.13 0.00 0.0132053 rpy=0 0 0
- joint left_pris1: limit lower=0.0 upper=0.0451 effort=0.0 velocity=0.0 -> lower=-0.0451 upper=0.0 effort=0.0 velocity=0.0
- joint rev2: axis 0 0 1 -> 0 0 -1; origin xyz=0.0 -0.02975 0.04475 rpy=-1.5707963267948968 1.5707963267948966 0 -> xyz=0.0 -0.02975 0.04475 rpy=-1.5707963267948968 1.5707963267948966 0.0
- joint rev3: axis 0 0 1 -> 0 0 -1
- joint rev5: axis 0 0 1 -> 0 0 -1
- joint rev7: axis 0 0 1 -> 0 0 -1
- joint right_pris2: limit lower=0.0 upper=0.0451 effort=0.0 velocity=0.0 -> lower=-0.0451 upper=0.0 effort=0.0 velocity=0.0
