Commit message: Add updated urdfs

File: openarm_bimanual_description/urdf/openarm_bimanual.urdf (robot description, URDF)
Before this commit: robot openarm_bimanual, 26 links, 25 joints
Links:
- added link camera_accel_frame
- added link camera_accel_optical_frame
- added link camera_bottom_screw_frame
- added link camera_color_frame
- added link camera_color_optical_frame
- added link camera_depth_frame
- added link camera_depth_optical_frame
- added link camera_gyro_frame
- added link camera_gyro_optical_frame
- added link camera_infra1_frame
- added link camera_infra1_optical_frame
- added link camera_infra2_frame
- added link camera_infra2_optical_frame
- added link camera_link, mass 0.072; collision box size=0.02505 0.09 0.025; visual mesh filename=file:///opt/ros/humble/share/realsense2_description/meshes/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
Joints:
- added joint camera_accel_joint: type fixed, parent camera_link, child camera_accel_frame, origin xyz=-0.01174 -0.00552 0.0051 rpy=0 0 0
- added joint camera_accel_optical_joint: type fixed, parent camera_accel_frame, child camera_accel_optical_frame, origin xyz=0 0 0 rpy=-1.5707963267948966 0 -1.5707963267948966
- added joint camera_color_joint: type fixed, parent camera_link, child camera_color_frame, origin xyz=0 0.015 0 rpy=0 0 0
- added joint camera_color_optical_joint: type fixed, parent camera_color_frame, child camera_color_optical_frame, origin xyz=0 0 0 rpy=-1.5707963267948966 0 -1.5707963267948966
- added joint camera_depth_joint: type fixed, parent camera_link, child camera_depth_frame, origin xyz=0 0 0 rpy=0 0 0
- added joint camera_depth_optical_joint: type fixed, parent camera_depth_frame, child camera_depth_optical_frame, origin xyz=0 0 0 rpy=-1.5707963267948966 0 -1.5707963267948966
- added joint camera_gyro_joint: type fixed, parent camera_link, child camera_gyro_frame, origin xyz=-0.01174 -0.00552 0.0051 rpy=0 0 0
- added joint camera_gyro_optical_joint: type fixed, parent camera_gyro_frame, child camera_gyro_optical_frame, origin xyz=0 0 0 rpy=-1.5707963267948966 0 -1.5707963267948966
- added joint camera_infra1_joint: type fixed, parent camera_link, child camera_infra1_frame, origin xyz=0 0.0 0 rpy=0 0 0
- added joint camera_infra1_optical_joint: type fixed, parent camera_infra1_frame, child camera_infra1_optical_frame, origin xyz=0 0 0 rpy=-1.5707963267948966 0 -1.5707963267948966
- added joint camera_infra2_joint: type fixed, parent camera_link, child camera_infra2_frame, origin xyz=0 -0.05 0 rpy=0 0 0
- added joint camera_infra2_optical_joint: type fixed, parent camera_infra2_frame, child camera_infra2_optical_frame, origin xyz=0 0 0 rpy=-1.5707963267948966 0 -1.5707963267948966
- added joint camera_joint: type fixed, parent pedestal_link, child camera_bottom_screw_frame, origin xyz=0.0 -0.025 0.995216 rpy=0.0 1.3962634015954636 -1.5707963267948966
- added joint camera_link_joint: type fixed, parent camera_bottom_screw_frame, child camera_link, origin xyz=0.010600000000000002 0.0175 0.0125 rpy=0 0 0
- joint left_left_pris1: axis 0 0 1 -> 0 0 -1; limit lower=-0.0451 upper=0.0 effort=0.0 velocity=0.0 -> lower=-0.0451 upper=0.0 effort=0.0 velocity=0.1
- joint left_rev2: limit lower=0.0 upper=3.141592653589793 effort=0.0 velocity=0.0 -> lower=0 upper=3.141592653589793 effort=0.0 velocity=0.0
- joint left_rev3: limit lower=-3.6651914291880923 upper=0.5235987755982988 effort=0.0 velocity=0.0 -> lower=-3.66519 upper=0.52359 effort=0.0 velocity=0.0
- joint left_right_pris2: axis 0 0 1 -> 0 0 -1
- joint right_left_pris1: axis 0 0 1 -> 0 0 -1; limit lower=-0.0451 upper=0.0 effort=0.0 velocity=0.0 -> lower=-0.0451 upper=0.0 effort=0.0 velocity=0.1
- joint right_rev2: axis 0 0 -1 -> 0 0 1; limit lower=-3.141592653589793 upper=0 effort=0.0 velocity=0.0 -> lower=0 upper=3.141592653589793 effort=0.0 velocity=0.0
- joint right_rev3: limit lower=-3.6651914291880923 upper=0.5235987755982988 effort=0.0 velocity=0.0 -> lower=-0.52359 upper=3.66519 effort=0.0 velocity=0.0
- joint right_right_pris2: axis 0 0 1 -> 0 0 -1

File: openarm_description/urdf/openarm.urdf (robot description, URDF)
Before this commit: robot openarm, 12 links, 11 joints
Joints:
- joint left_pris1: axis 0 0 1 -> 0 0 -1; limit lower=-0.0451 upper=0.0 effort=0.0 velocity=0.0 -> lower=-0.0451 upper=0.0 effort=0.0 velocity=0.1
- joint rev2: axis 0 0 -1 -> 0 0 1
- joint rev3: limit lower=-3.6651914291880923 upper=0.5235987755982988 effort=0.0 velocity=0.0 -> lower=-0.52359 upper=3.66519 effort=0.0 velocity=0.0
- joint right_pris2: axis 0 0 1 -> 0 0 -1

Commit message: Update generated urdfs

File: openarm_bimanual_description/urdf/openarm_bimanual.urdf (robot description, URDF)
Before this commit: robot openarm_bimanual, 40 links, 39 joints
Joints:
- joint left_rev1: limit lower=-2.0943951023931953 upper=2.0943951023931953 effort=0.0 velocity=0.0 -> lower=-2.0943951023931953 upper=0.7853981633974483 effort=0.0 velocity=0.0
- joint left_rev2: limit lower=0 upper=3.141592653589793 effort=0.0 velocity=0.0 -> lower=-0.17453292519943295 upper=2.9670597283903604 effort=0.0 velocity=0.0
- joint left_rev3: limit lower=-3.66519 upper=0.52359 effort=0.0 velocity=0.0 -> lower=-2.0943951023931953 upper=2.0943951023931953 effort=0.0 velocity=0.0
- joint left_rev4: limit lower=-0.3490658503988659 upper=2.792526803190927 effort=0.0 velocity=0.0 -> lower=0 upper=2.6179938779914944 effort=0.0 velocity=0.0
- joint left_rev7: limit lower=-0.9599310885968813 upper=0.9599310885968813 effort=0.0 velocity=0.0 -> lower=-0.9599310885968811 upper=0.9599310885968811 effort=0.0 velocity=0.0
- joint right_rev1: limit lower=-2.0943951023931953 upper=2.0943951023931953 effort=0.0 velocity=0.0 -> lower=-0.7853981633974483 upper=2.0943951023931953 effort=0.0 velocity=0.0
- joint right_rev2: limit lower=0 upper=3.141592653589793 effort=0.0 velocity=0.0 -> lower=-0.17453292519943295 upper=2.9670597283903604 effort=0.0 velocity=0.0
- joint right_rev3: limit lower=-0.52359 upper=3.66519 effort=0.0 velocity=0.0 -> lower=-2.0943951023931953 upper=2.0943951023931953 effort=0.0 velocity=0.0
- joint right_rev4: limit lower=-0.3490658503988659 upper=2.792526803190927 effort=0.0 velocity=0.0 -> lower=0 upper=2.6179938779914944 effort=0.0 velocity=0.0
- joint right_rev7: limit lower=-0.9599310885968813 upper=0.9599310885968813 effort=0.0 velocity=0.0 -> lower=-0.9599310885968811 upper=0.9599310885968811 effort=0.0 velocity=0.0

File: openarm_description/urdf/openarm.urdf (robot description, URDF)
Before this commit: robot openarm, 12 links, 11 joints
Joints:
- joint rev3: limit lower=-0.52359 upper=3.66519 effort=0.0 velocity=0.0 -> lower=-2.0943951023931953 upper=2.0943951023931953 effort=0.0 velocity=0.0
- joint rev4: limit lower=-0.3490658503988659 upper=2.792526803190927 effort=0.0 velocity=0.0 -> lower=0 upper=2.6179938779914944 effort=0.0 velocity=0.0
- joint rev7: limit lower=-0.9599310885968813 upper=0.9599310885968813 effort=0.0 velocity=0.0 -> lower=-0.9599310885968811 upper=0.9599310885968811 effort=0.0 velocity=0.0

Commit message: Add mujoco ros2 control (#26)
Add support for simulated openarm hardware with MuJoCo backend.

File: openarm_bimanual_description/urdf/openarm_bimanual.urdf (robot description, URDF)
Before this commit: robot openarm_bimanual, 40 links, 39 joints
Joints:
- removed joint left_left_pris1
- removed joint left_right_pris2
- removed joint right_left_pris1
- removed joint right_right_pris2
- added joint left_gripper: type prismatic, parent left_link8, child left_link_left_jaw, origin xyz=-0.1071 0.0768568 0.0132053 rpy=1.570796326795101 -0.014066001454929162 0.00875904933542146, axis 0 0 -1, limit lower=-0.0451 upper=0.0 effort=0.0 velocity=0.1
- added joint left_gripper_mimic: type prismatic, parent left_link8, child left_link_right_jaw, origin xyz=-0.10571 -0.0781373 0.0132053 rpy=1.570796326794883 -0.014066001454927403 0.008759049336290027, axis 0 0 -1, limit lower=-0.0451 upper=0.0 effort=0.0 velocity=0.0, mimic joint=left_gripper multiplier=-1.0 offset=0.0
- added joint right_gripper: type prismatic, parent right_link8, child right_link_left_jaw, origin xyz=-0.1071 0.0768568 0.0132053 rpy=1.570796326795101 -0.014066001454929162 0.00875904933542146, axis 0 0 -1, limit lower=-0.0451 upper=0.0 effort=0.0 velocity=0.1
- added joint right_gripper_mimic: type prismatic, parent right_link8, child right_link_right_jaw, origin xyz=-0.10571 -0.0781373 0.0132053 rpy=1.570796326794883 -0.014066001454927403 0.008759049336290027, axis 0 0 -1, limit lower=-0.0451 upper=0.0 effort=0.0 velocity=0.0, mimic joint=right_gripper multiplier=-1.0 offset=0.0

File: openarm_bimanual_description/urdf/openarm_bimanual.urdf.xacro (robot description, xacro)
@@ -13,4 +13,5 @@
 -->
 <robot xmlns:xacro="http://www.ros.org/wiki/xacro" name="openarm_bimanual">
+  <xacro:arg name="hardware_type" default="real" />
   <!-- Robot description parameters -->
   <xacro:arg name="prefix" default="" />
@@ -18,5 +19,5 @@
   <xacro:arg name="right_can_device" default="can0" />
   <xacro:arg name="left_can_device" default="can1" />
-  <xacro:arg name="use_mock_hardware" default="false" />
+  <xacro:arg name="hardware_type" default="real" />
   <xacro:arg name="mock_sensor_commands" default="false" />
   <xacro:include filename="$(find openarm_description)/urdf/openarm.robot.xacro"/>
@@ -45,5 +46,5 @@
   <xacro:arg name="right_initial_positions_file" default="$(find openarm_description)/config/initial_positions.yaml" />
   <xacro:arg name="left_initial_positions_file" default="$(find openarm_description)/config/initial_positions.yaml" />
-  <xacro:openarm_ros2_control name="RightOpenArmHW" prefix="right_" initial_positions_file="$(arg right_initial_positions_file)" can_device="$(arg right_can_device)" use_mock_hardware="$(arg use_mock_hardware)" mock_sensor_commands="$(arg mock_sensor_commands)"/>
-  <xacro:openarm_ros2_control name="LeftOpenArmHW" prefix="left_" initial_positions_file="$(arg left_initial_positions_file)" can_device="$(arg left_can_device)" use_mock_hardware="$(arg use_mock_hardware)" mock_sensor_commands="$(arg mock_sensor_commands)"/>
+  <xacro:openarm_ros2_control name="RightOpenArmHW" prefix="right_" initial_positions_file="$(arg right_initial_positions_file)" can_device="$(arg right_can_device)" hardware_type="$(arg hardware_type)" mock_sensor_commands="$(arg mock_sensor_commands)"/>
+  <xacro:openarm_ros2_control name="LeftOpenArmHW" prefix="left_" initial_positions_file="$(arg left_initial_positions_file)" can_device="$(arg left_can_device)" hardware_type="$(arg hardware_type)" mock_sensor_commands="$(arg mock_sensor_commands)"/>
 </robot>

File: openarm_description/urdf/openarm.robot.xacro (robot description, xacro)
@@ -25,4 +25,5 @@
         <xacro:property name="reflect" value="${1 if side=='right' else -1}"/>
         <xacro:property name="rotate" value="${0 if side=='right' else pi}"/>
+        <!-- ros2_control configuration is handled separately in openarm.urdf.xacro -->
         <link name="${prefix}dummy_link"/>
         <joint name="${prefix}dummy_joint" type="fixed">
@@ -280,5 +281,6 @@
             <limit effort="0.0" lower="${-pi * 11.0 / 36.0}" upper="${pi * 11.0 / 36.0}" velocity="0.0"/>
         </joint>
-        <joint name="${prefix}left_pris1" type="prismatic">
+        <!-- this is used as the actuator interface, the other gripper mimics motion -->
+        <joint name="${prefix}gripper" type="prismatic">
             <parent link="${prefix}link8"/>
             <child link="${prefix}link_left_jaw"/>
@@ -287,5 +289,5 @@
             <limit effort="0.0" lower="-0.0451" upper="0.0" velocity="0.1"/>
         </joint>
-        <joint name="${prefix}right_pris2" type="prismatic">
+        <joint name="${prefix}gripper_mimic" type="prismatic">
             <parent link="${prefix}link8"/>
             <child link="${prefix}link_right_jaw"/>
@@ -293,5 +295,5 @@
             <axis xyz="0 0 -1"/>
             <limit effort="0.0" lower="-0.0451" upper="0.0" velocity="0.0"/>
-            <mimic joint="${prefix}left_pris1" multiplier="-1.0" offset="0.0"/>
+            <mimic joint="${prefix}gripper" multiplier="-1.0" offset="0.0"/>
         </joint>
         <joint name="${prefix}virtual_gripper_center" type="fixed">

File: openarm_description/urdf/openarm.ros2_control.xacro (robot description, xacro)
@@ -13,79 +13,98 @@
 -->
 <robot xmlns:xacro="http://www.ros.org/wiki/xacro">
-    <xacro:macro name="openarm_ros2_control" params="name initial_positions_file prefix:='' can_device='can0' use_mock_hardware:=false mock_sensor_commands:=false">
+    <xacro:macro name="openarm_ros2_control" params="name initial_positions_file websocket_port='' prefix:='' can_device='can0' hardware_type='real' mock_sensor_commands='{}'">
         <xacro:property name="initial_positions" value="${xacro.load_yaml(initial_positions_file)['initial_positions']}"/>
+        <!-- Set default websocket ports based on prefix if not provided -->
+        <xacro:if value="${hardware_type == 'sim' and websocket_port == ''}">
+            <xacro:property name="computed_websocket_port" value="${'1337' if prefix == 'right_' or prefix == '' else '1338'}"/>
+        </xacro:if>
+        <xacro:unless value="${hardware_type == 'sim' and websocket_port == ''}">
+            <xacro:property name="computed_websocket_port" value="${websocket_port}"/>
+        </xacro:unless>
         <ros2_control name="${prefix}${name}" type="system">
             <hardware>
-                <xacro:if value="${use_mock_hardware}">
+                <xacro:if value="${hardware_type == 'mock'}">
                     <plugin>mock_components/GenericSystem</plugin>
                     <param name="mock_sensor_commands">${mock_sensor_commands}</param>
                 </xacro:if>
-                <xacro:unless value="${use_mock_hardware}">
+                <xacro:if value="${hardware_type == 'sim'}">
+                    <plugin>openarm_mujoco_hardware/MujocoHardware</plugin>
+                    <param name="prefix">${prefix}</param>
+                    <xacro:if value="${computed_websocket_port != ''}">
+                        <param name="websocket_port">${computed_websocket_port}</param>
+                    </xacro:if>
+                </xacro:if>
+                <xacro:if value="${hardware_type == 'real'}">
                     <plugin>openarm_hardware/OpenArmHW</plugin>
                     <param name="prefix">${prefix}</param>
                     <param name="can_device">${can_device}</param>
-                </xacro:unless>
+                </xacro:if>
             </hardware>
             <joint name="${prefix}rev1">
                 <command_interface name="position"/>
                 <command_interface name="velocity"/>
-                <command_interface name="effort"/>
+                <!-- <command_interface name="effort"/> -->
                 <state_interface name="position"/>
                 <state_interface name="velocity"/>
-                <state_interface name="effort"/>
+                <!-- <state_interface name="effort"/> -->
             </joint>
             <joint name="${prefix}rev2">
                 <command_interface name="position"/>
                 <command_interface name="velocity"/>
-                <command_interface name="effort"/>
+                <!-- <command_interface name="effort"/> -->
                 <state_interface name="position"/>
                 <state_interface name="velocity"/>
-                <state_interface name="effort"/>
+                <!-- <state_interface name="effort"/> -->
             </joint>
             <joint name="${prefix}rev3">
                 <command_interface name="position"/>
                 <command_interface name="velocity"/>
-                <command_interface name="effort"/>
+                <!-- <command_interface name="effort"/> -->
                 <state_interface name="position"/>
                 <state_interface name="velocity"/>
-                <state_interface name="effort"/>
+                <!-- <state_interface name="effort"/> -->
             </joint>
             <joint name="${prefix}rev4">
                 <command_interface name="position"/>
                 <command_interface name="velocity"/>
-                <command_interface name="effort"/>
+                <!-- <command_interface name="effort"/> -->
                 <state_interface name="position"/>
                 <state_interface name="velocity"/>
-                <state_interface name="effort"/>
+                <!-- <state_interface name="effort"/> -->
             </joint>
             <joint name="${prefix}rev5">
                 <command_interface name="position"/>
                 <command_interface name="velocity"/>
-                <command_interface name="effort"/>
+                <!-- <command_interface name="effort"/> -->
                 <state_interface name="position"/>
                 <state_interface name="velocity"/>
-                <state_interface name="effort"/>
+                <!-- <state_interface name="effort"/> -->
             </joint>
             <joint name="${prefix}rev6">
                 <command_interface name="position"/>
                 <command_interface name="velocity"/>
-                <command_interface name="effort"/>
+                <!-- <command_interface name="effort"/> -->
                 <state_interface name="position"/>
                 <state_interface name="velocity"/>
-                <state_interface name="effort"/>
+                <!-- <state_interface name="effort"/> -->
             </joint>
             <joint name="${prefix}rev7">
                 <command_interface name="position"/>
                 <command_interface name="velocity"/>
-                <command_interface name="effort"/>
+                <!-- <command_interface name="effort"/> -->
                 <state_interface name="position"/>
                 <state_interface name="velocity"/>
-                <state_interface name="effort"/>
+                <!-- <state_interface name="effort"/> -->
             </joint>
-            <joint name="${prefix}left_pris1">
+            <joint name="${prefix}gripper">
                 <command_interface name="position"/>
                 <state_interface name="position"/>
                 <state_interface name="velocity"/>
             </joint>
+            <!-- <joint name="${prefix}gripper_mimic">
+                <state_interface name="position">
+                  <param name="initial_value">${initial_positions['gripper_mimic']}</param>
+                </state_interface>
+            </joint> -->
         </ros2_control>
     </xacro:macro>

File: openarm_description/urdf/openarm.urdf (robot description, URDF)
Before this commit: robot openarm, 12 links, 11 joints
Joints:
- removed joint left_pris1
- removed joint right_pris2
- added joint gripper: type prismatic, parent link8, child link_left_jaw, origin xyz=-0.1071 0.0768568 0.0132053 rpy=1.570796326795101 -0.014066001454929162 0.00875904933542146, axis 0 0 -1, limit lower=-0.0451 upper=0.0 effort=0.0 velocity=0.1
- added joint gripper_mimic: type prismatic, parent link8, child link_right_jaw, origin xyz=-0.10571 -0.0781373 0.0132053 rpy=1.570796326794883 -0.014066001454927403 0.008759049336290027, axis 0 0 -1, limit lower=-0.0451 upper=0.0 effort=0.0 velocity=0.0, mimic joint=gripper multiplier=-1.0 offset=0.0
